File: board-prototype/control.sch (KiCad schematic (older format))
At the start: 18 parts, among them U115 74LVC7T245, U116 74LVC7T245, U117 74LVC7T245, U118 74LVC7T245, U119 74LVC7T245, U201 DS8641-LR, U202 DS8641-LR, U203 DS8641-LR, U204 DS8641-LR, U205 DS8641-LR

Commit message: Changed over to only DS8641 bus transceivers and the smaller package level-converters.
Parts:
- removed U115, U116, U117, U118, U119: 74LVC7T245, SMD_Packages:SOIC-24, symbol 74LVC7T245
- added U115, U116, U117, U118, U119: 74LVC8T245, Housings_SSOP:TSSOP-24_4.4x7.8mm_Pitch0.65mm, symbol 74LVC8T245
Connections:
- net +3V3: now also U115.23 (VCCb), U115.24 (VCCb), U116.1 (VCCa), U117.23 (VCCb), U117.24 (VCCb), U118.1 (VCCa), U119.1 (VCCa)
- net +5V: now also U115.1 (VCCa), U116.23 (VCCb), U116.24 (VCCb), U117.1 (VCCa), U118.23 (VCCb), U118.24 (VCCb), U119.23 (VCCb), U119.24 (VCCb)
- net BDCOK: now also U205.1 (bus3); no longer U205.12 (bus2)
- net BIRQ7: now also U205.12 (bus2); no longer U205.4 (bus4)
- net BPOK: now also U205.4 (bus4); no longer U205.15 (bus1)
- net BSACK: now also U205.15 (bus1); no longer U205.1 (bus3)
- net GND: now also U205.2 (in3), U205.5 (in4), U115.11 (GND), U115.12 (GND), U115.13 (GND), U115.2 (A->B), U115.22 (~OE), U116.11 (GND), U116.12 (GND), U116.13 (GND), U116.2 (A->B), U116.22 (~OE), U117.11 (GND), U117.12 (GND), U117.13 (GND), U117.2 (A->B), U117.22 (~OE), U118.11 (GND), U118.12 (GND), U118.13 (GND), U118.2 (A->B), U118.22 (~OE), U119.11 (GND), U119.12 (GND), U119.13 (GND), U119.2 (A->B), U119.22 (~OE); no longer U205.11 (in2), U205.14 (in1)
- net RDCOK: now also U119.5 (A2)
- net RDIN: now also U116.8 (A5)
- net RDMGI: now also U118.6 (A3)
- net RDMR: now also U118.4 (A1)
- net RDOUT: now also U116.5 (A2)
- net RHALT: now also U118.8 (A5)
- net RIAKI: now also U116.10 (A7)
- net RINIT: now also U118.10 (A7)
- net RIRQ4: now also U116.9 (A6)
- net RIRQ5: now also U116.3 (A0)
- net RIRQ6: now also U116.4 (A1)
- net RIRQ7: now also U119.4 (A1)
- net RPOK: now also U119.6 (A3)
- net RREF: now also U118.5 (A2)
- net RRPLY: now also U116.6 (A3)
- net RSACK: now also U119.3 (A0)
- net RSYNC: now also U116.7 (A4)
- net TDIN: now also U115.16 (B5)
- net TDMGO: now also U117.16 (B5)
- net TDMR: now also U117.20 (B1)
- net TDOUT: now also U115.19 (B2)
- net TIAKO: now also U117.21 (B0)
- net TIRQ4: now also U115.15 (B6)
- net TIRQ5: now also U115.21 (B0)
- net TIRQ6: now also U115.20 (B1)
- net TIRQ7: now also U117.15 (B6)
- net TREF: now also U117.19 (B2)
- net TRPLY: now also U115.18 (B3)
- net TSACK: now also U117.17 (B4)
- net TSYNC: now also U115.17 (B4)
- net at U201.14 (in1): now also U115.3 (A0)
- net at U201.11 (in2): now also U115.4 (A1)
- net at U201.2 (in3): now also U115.5 (A2)
- net at U201.5 (in4): now also U115.6 (A3)
- net at U202.14 (in1): now also U115.7 (A4)
- net at U202.11 (in2): now also U115.8 (A5)
- net at U202.2 (in3): now also U115.9 (A6)
- net at U202.6 (out4): now also U116.14 (B7)
- net at U202.3 (out3): now also U116.15 (B6)
- net at U202.10 (out2): now also U116.16 (B5)
- net at U202.13 (out1): now also U116.17 (B4)
- net at U201.6 (out4): now also U116.18 (B3)
- net at U201.3 (out3): now also U116.19 (B2)
- net at U201.10 (out2): now also U116.20 (B1)
- net at U201.13 (out1): now also U116.21 (B0)
- net at U203.14 (in1): now also U117.3 (A0)
- net at U203.11 (in2): now also U117.4 (A1)
- net at U203.2 (in3): now also U117.5 (A2)
- net at U204.14 (in1): now also U117.8 (A5)
- net at U204.6 (out4): now also U118.14 (B7)
- net at U204.10 (out2): now also U118.16 (B5)
- net at U203.6 (out4): now also U118.18 (B3)
- net at U203.3 (out3): now also U118.19 (B2)
- net at U203.10 (out2): now also U118.20 (B1)
- net at U205.6 (out4): now also U119.18 (B3)
- net at U205.3 (out3): now also U119.19 (B2)
- net at U205.10 (out2): now also U119.20 (B1)
- net at U205.13 (out1): now also U119.21 (B0)
- new net: U117.9 (A6), U205.11 (in2)
- new net: U117.7 (A4), U205.14 (in1)

Commit message: Updated to KiCad 5
Parts:
- R101, R102, R103, R104, R105, R106, R107, R108: symbol R -> device:R
- U115, U116, U117, U118, U119: symbol 74LVC8T245 -> myLib:74LVC8T245
- U201, U202, U203, U204, U205: symbol DS8641-LR -> myLib:DS8641-LR
Changed lines of the file:
@@
-EESchema Schematic File Version 2
-LIBS:power
-LIBS:device
-LIBS:transistors
-LIBS:conn
-LIBS:linear
-LIBS:regul
-LIBS:74xx
-LIBS:cmos4000
-LIBS:adc-dac
-LIBS:memory
-LIBS:xilinx
-LIBS:microcontrollers
-LIBS:dsp
-LIBS:microchip
-LIBS:analog_switches
-LIBS:motorola
-LIBS:texas
-LIBS:intel
-LIBS:audio
-LIBS:interface
-LIBS:digital-audio
-LIBS:philips
-LIBS:display
-LIBS:cypress
-LIBS:siliconi
-LIBS:opto
-LIBS:atmel
-LIBS:contrib
-LIBS:valves
-LIBS:myLib
+EESchema Schematic File Version 4
 LIBS:proto-cache
-EELAYER 25 0
+EELAYER 26 0
 EELAYER END
 $Descr USLetter 8500 11000 portrait
@@
 $EndDescr
 $Comp
-L +5V #PWR095
+L power:+5V #PWR095
 U 1 1 56BE84AB
 P 2400 2100
@@
 $EndComp
 $Comp
-L +3.3V #PWR096
+L power:+3.3V #PWR096
 U 1 1 56BE84B1
 P 2050 2100
@@
 $EndComp
 $Comp
-L +5V #PWR097
+L power:+5V #PWR097
 U 1 1 56BE84BE
 P 2400 4300
@@
 $EndComp
 $Comp
-L +3.3V #PWR098
+L power:+3.3V #PWR098
 U 1 1 56BE84C4
 P 2050 4300
@@
 $EndComp
 $Comp
-L +5V #PWR099
+L power:+5V #PWR099
 U 1 1 56BE84D0
 P 5750 2100
@@
 $EndComp
 $Comp
-L +3.3V #PWR0100
+L power:+3.3V #PWR0100
 U 1 1 56BE84D6
 P 6100 2100
@@
 $EndComp
 $Comp
-L +5V #PWR0101
+L power:+5V #PWR0101
 U 1 1 56BE84E9
 P 5750 4300
@@
 $EndComp
 $Comp
-L +3.3V #PWR0102
+L power:+3.3V #PWR0102
 U 1 1 56BE84EF
 P 6100 4300
@@
 NoConn ~ 6550 8600
 $Comp
-L GND #PWR0103
+L power:GND #PWR0103
 U 1 1 56BE8504
 P 6550 8950
@@
 $EndComp
 $Comp
-L +3.3V #PWR0104
+L power:+3.3V #PWR0104
 U 1 1 56BE850A
 P 6100 7650
@@
 $EndComp
 $Comp
-L +5V #PWR0105
+L power:+5V #PWR0105
 U 1 1 56BE8510
 P 5750 7650
@@
 NoConn ~ 5350 5150
 $Comp
-L DS8641-LR U201
+L myLib:DS8641-LR U201
 U 1 1 56BE854E
 P 4150 1450
@@
 $EndComp
 $Comp
-L DS8641-LR U202
+L myLib:DS8641-LR U202
 U 1 1 56BE8555
 P 4150 3050
@@
 $EndComp
 $Comp
-L DS8641-LR U203
+L myLib:DS8641-LR U203
 U 1 1 56BE855C
 P 4150 4850
@@
 $EndComp
 $Comp
-L DS8641-LR U204
+L myLib:DS8641-LR U204
 U 1 1 56BE8563
 P 4150 6450
@@
 $EndComp
 $Comp
-L DS8641-LR U205
+L myLib:DS8641-LR U205
 U 1 1 56BE856A
 P 4150 8200
@@
 $EndComp
 $Comp
-L GND #PWR0106
+L power:GND #PWR0106
 U 1 1 56BE8571
 P 3300 8150
@@
 $EndComp
 $Comp
-L GND #PWR0107
+L power:GND #PWR0107
 U 1 1 56BE8577
 P 3450 7700
@@
 NoConn ~ 6550 4550
 Wire Wire Line
-	6550 3250 6550 3400
+	6550 3250 6550 3350
 Connection ~ 6550 3350
 Wire Wire Line
 	5850 2100 5750 2100
 Wire Wire Line
-	6550 5450 6550 5600
+	6550 5450 6550 5550
 Connection ~ 6550 5550
 Wire Wire Line
 	5850 4300 5750 4300
 Wire Wire Line
-	6550 8800 6550 8950
+	6550 8800 6550 8900
 Connection ~ 6550 8900
 Wire Wire Line
@@
 	3450 6250 3400 6250
 Wire Wire Line
-	3400 6250 3400 6500
-$Comp
-L +5V #PWR0108
+	3400 6250 3400 6350
+$Comp
+L power:+5V #PWR0108
 U 1 1 56BE8D9E
 P 2250 8950
@@
 $EndComp
 $Comp
-L R R105
+L device:R R105
 U 1 1 56BE8DAA
 P 2250 9100
@@
 $EndComp
 $Comp
-L R R106
+L device:R R106
 U 1 1 56BE8DB1
 P 2250 9500
@@
 $EndComp
 $Comp
-L +5V #PWR0109
+L power:+5V #PWR0109
 U 1 1 56BE8DB8
 P 2850 8950
@@
 $EndComp
 $Comp
-L R R107
+L device:R R107
 U 1 1 56BE8DC4
 P 2850 9100
@@
 $EndComp
 $Comp
-L R R108
+L device:R R108
 U 1 1 56BE8DCB
 P 2850 9500
@@
 $EndComp
 $Comp
-L +5V #PWR0110
+L power:+5V #PWR0110
 U 1 1 56BE8DD2
 P 1100 8950
@@
 $EndComp
 $Comp
-L GND #PWR0111
+L power:GND #PWR0111
 U 1 1 56BE8DD8
 P 1100 9650
@@
 $EndComp
 $Comp
-L R R101
+L device:R R101
 U 1 1 56BE8DDE
 P 1100 9100
@@
 $EndComp
 $Comp
-L R R102
+L device:R R102
 U 1 1 56BE8DE5
 P 1100 9500
@@
 $EndComp
 $Comp
-L +5V #PWR0112
+L power:+5V #PWR0112
 U 1 1 56BE8DED
 P 1700 8950
@@
 $EndComp
 $Comp
-L R R103
+L device:R R103
 U 1 1 56BE8DF9
 P 1700 9100
@@
 $EndComp
 $Comp
-L R R104
+L device:R R104
 U 1 1 56BE8E00
 P 1700 9500
@@
 $EndComp
 Wire Wire Line
-	2250 9250 2250 9350
+	2250 9250 2250 9300
 Wire Wire Line
 	2250 9300 2300 9300
 Connection ~ 2250 9300
 Wire Wire Line
-	2850 9250 2850 9350
+	2850 9250 2850 9300
 Wire Wire Line
 	2850 9300 2900 9300
 Connection ~ 2850 9300
 Wire Wire Line
-	1100 9250 1100 9350
+	1100 9250 1100 9300
 Wire Wire Line
 	1100 9300 1150 9300
 Connection ~ 1100 9300
 Wire Wire Line
-	1700 9250 1700 9350
+	1700 9250 1700 9300
 Wire Wire Line
 	1700 9300 1750 9300
@@
 BIAKO
 $Comp
-L GND #PWR0113
+L power:GND #PWR0113
 U 1 1 56CE07FC
 P 1700 9650
@@
 $EndComp
 $Comp
-L GND #PWR0114
+L power:GND #PWR0114
 U 1 1 56CE083D
 P 2250 9650
@@
 $EndComp
 $Comp
-L GND #PWR0115
+L power:GND #PWR0115
 U 1 1 56CE087E
 P 2850 9650
@@
 $EndComp
 $Comp
-L GND #PWR0116
+L power:GND #PWR0116
 U 1 1 56CE0C91
 P 3400 6500
@@
 $EndComp
 $Comp
-L GND #PWR0117
+L power:GND #PWR0117
 U 1 1 56CE0D99
 P 3450 5950
@@
 $EndComp
 $Comp
-L GND #PWR0118
+L power:GND #PWR0118
 U 1 1 56CE0DED
 P 2850 5550
@@
 $EndComp
 $Comp
-L GND #PWR0119
+L power:GND #PWR0119
 U 1 1 56CE0FD0
 P 3450 4850
@@
 $EndComp
 $Comp
-L GND #PWR0120
+L power:GND #PWR0120
 U 1 1 56CE1011
 P 3450 4350
@@
 $EndComp
 $Comp
-L GND #PWR0121
+L power:GND #PWR0121
 U 1 1 56CE10D1
 P 6550 5600
@@
 $EndComp
 $Comp
-L GND #PWR0122
+L power:GND #PWR0122
 U 1 1 56CE11B5
 P 6550 3400
@@
 $EndComp
 $Comp
-L GND #PWR0123
+L power:GND #PWR0123
 U 1 1 56CE1313
 P 3450 3050
@@
 $EndComp
 $Comp
-L GND #PWR0124
+L power:GND #PWR0124
 U 1 1 56CE1354
 P 3450 2550
@@
 $EndComp
 $Comp
-L GND #PWR0125
+L power:GND #PWR0125
 U 1 1 56CE1395
 P 2850 3350
@@
 $EndComp
 $Comp
-L GND #PWR0126
+L power:GND #PWR0126
 U 1 1 56CE151B
 P 3450 950
@@
 $EndComp
 $Comp
-L 74LVC8T245 U116
+L myLib:74LVC8T245 U116
 U 1 1 580E306F
 P 5950 2850
@@
 $EndComp
 $Comp
-L 74LVC8T245 U118
+L myLib:74LVC8T245 U118
 U 1 1 580E30E9
 P 5950 5050
@@
 $EndComp
 $Comp
-L 74LVC8T245 U119
+L myLib:74LVC8T245 U119
 U 1 1 580E3161
 P 5950 8400
@@
 $EndComp
 $Comp
-L 74LVC8T245 U115
+L myLib:74LVC8T245 U115
 U 1 1 580E31E0
 P 2250 2850
@@
 $EndComp
 $Comp
-L 74LVC8T245 U117
+L myLib:74LVC8T245 U117
 U 1 1 580E325A
 P 2250 5050
@@
 $EndComp
 Wire Wire Line
-	3450 8100 3450 8200
+	3450 8100 3450 8150
 Wire Wire Line
 	3300 8150 3450 8150
@@
 Wire Wire Line
 	3100 5150 2850 5150
+Wire Wire Line
+	6550 3350 6550 3400
+Wire Wire Line
+	6550 5550 6550 5600
+Wire Wire Line
+	6550 8900 6550 8950
+Wire Wire Line
+	3400 6350 3400 6450
+Wire Wire Line
+	3400 6450 3400 6500
+Wire Wire Line
+	2250 9300 2250 9350
+Wire Wire Line
+	2850 9300 2850 9350
+Wire Wire Line
+	1100 9300 1100 9350
+Wire Wire Line
+	1700 9300 1700 9350
+Wire Wire Line
+	3450 8150 3450 8200
 $EndSCHEMATC
