File: board-prototype/fpga.sch (KiCad schematic (older format))
At the start: 9 parts, among them P1 AB, P101 Data, P102 Power, P103 Logic Analyzer, P2 CD, SW401 RESET, U110 MAX3488, U111 MAX3488, U112 MAX3488

Commit message: Changed over to only DS8641 bus transceivers and the smaller package level-converters.
Parts:
- removed P101: Data, Pin_Headers:Pin_Header_Angled_2x04, symbol CONN_02X04
- removed P102: Power, Pin_Headers:Pin_Header_Angled_2x05, symbol CONN_02X05
- removed SW401: RESET, symbol SW_PUSH_SMALL
- removed U110, U111, U112: MAX3488, Housings_SOIC:SOIC-8_3.9x4.9mm_Pitch1.27mm, symbol MAX3488
- added P101: Data, Pin_Headers:Pin_Header_Angled_2x05, symbol CONN_02X05
- added P102: Power, Pin_Headers:Pin_Header_Angled_2x04, symbol CONN_02X04
- added U401: MAX3033E, Housings_SOIC:SOIC-16_3.9x9.9mm_Pitch1.27mm, symbol MAX3033E
- P103: footprint Socket_Strips:Socket_Strip_Straight_2x16 -> Pin_Headers:Pin_Header_Straight_2x16
Connections:
- net +12V: now also P102.3 (P3), P102.4 (P4), P102.5 (P5), P102.6 (P6)
- net GND: now also P102.1 (P1), P102.2 (P2), P102.7 (P7), P102.8 (P8), U401.8 (GND)
- net IPclk: now also U401.1 (I1)
- net IPdata: now also U401.7 (I2)
- net IPlatch: now also U401.9 (I3)
- net RDAL3: now reaches P1.11 (A6)
- net TDAL6: now reaches P1.18 (B9)
- net TDAL7: now reaches P1.20 (B10)
- net TDAL8: now reaches P1.22 (B11)
- net RDAL13: now reaches P1.37 (A19)
- net TDAL12: now reaches P1.38 (B19)
- net RDAL16: now reaches P1.43 (A22)
- net TDAL15: now reaches P1.44 (B22)
- net RDAL0: now reaches P1.5 (A3)
- net TDAL18: now reaches P1.50 (B25)
- net TDAL19: now reaches P1.52 (B26)
- net TDAL20: now reaches P1.54 (B27)
- net TDAL21: now reaches P1.56 (B28)
- net RBS7: now reaches P1.57 (A29)
- net TBS7: now reaches P1.58 (B29)
- net RWTBT: now reaches P1.59 (A30)
- net TDAL0: now reaches P1.6 (B3)
- net TWTBT: now reaches P1.60 (B30)
- net RDAL1: now reaches P1.7 (A4)
- net TDAL1: now reaches P1.8 (B4)
- net RDAL2: now reaches P1.9 (A5)
- net DALst renamed RDAL20
- net DALtx renamed RDAL19
- net ZBS7 renamed RDAL18
- net ZDAL0 renamed TDAL2
- net ZDAL1 renamed TDAL3
- net ZDAL10 renamed RDAL10
- net ZDAL11 renamed TDAL9
- net ZDAL12 renamed RDAL11
- net ZDAL13 renamed TDAL10
- net ZDAL14 renamed RDAL12
- net ZDAL15 renamed TDAL11
- net ZDAL16 renamed RDAL14
- net ZDAL17 renamed TDAL13
- net ZDAL18 renamed RDAL15
- net ZDAL19 renamed TDAL14
- net ZDAL2 renamed RDAL4
- net ZDAL20 renamed RDAL17
- net ZDAL21 renamed TDAL16
- net ZDAL3 renamed TDAL4
- net ZDAL4 renamed RDAL5
- net ZDAL5 renamed TDAL5
- net ZDAL6 renamed RDAL6
- net ZDAL7 renamed RDAL7
- net ZDAL8 renamed RDAL8
- net ZDAL9 renamed RDAL9
- net ZWTBT renamed TDAL17
- net ~DALbe renamed RDAL21
- new net +3V3: U401.12 (EN34), U401.4 (EN12)
- new net IPblank_N: P101.10 (P10), U401.13 (O4-)
- new net IPblank_P: P101.9 (P9), U401.14 (O4+)
- new net IPclk_N: P101.8 (P8), U401.3 (O1-)
- new net IPclk_P: P101.7 (P7), U401.2 (O1+)
- new net IPdata_N: P101.4 (P4), U401.5 (O2-)
- new net IPdata_P: P101.3 (P3), U401.6 (O2+)
- new net IPlatch_N: P101.2 (P2), U401.11 (O3-)
- new net IPlatch_P: P101.1 (P1), U401.10 (O3+)
- new net VDD: U401.16 (VDD)
- new net ~IPblank: U401.15 (I4)
- no-connect marks 40 -> 33

Commit message: Updated to KiCad 5
Parts:
- P1: symbol CONN_ZTEX_AB -> myLib:CONN_ZTEX_AB
- P101: symbol CONN_02X05 -> conn:CONN_02X05
- P102: symbol CONN_02X04 -> conn:CONN_02X04
- P103: symbol CONN_02X16 -> conn:CONN_02X16
- P2: symbol CONN_ZTEX_CD -> myLib:CONN_ZTEX_CD
- U401: symbol MAX3033E -> proto-rescue:MAX3033E
Changed lines of the file:
@@
-EESchema Schematic File Version 2
-LIBS:power
-LIBS:device
-LIBS:transistors
-LIBS:conn
-LIBS:linear
-LIBS:regul
-LIBS:74xx
-LIBS:cmos4000
-LIBS:adc-dac
-LIBS:memory
-LIBS:xilinx
-LIBS:microcontrollers
-LIBS:dsp
-LIBS:microchip
-LIBS:analog_switches
-LIBS:motorola
-LIBS:texas
-LIBS:intel
-LIBS:audio
-LIBS:interface
-LIBS:digital-audio
-LIBS:philips
-LIBS:display
-LIBS:cypress
-LIBS:siliconi
-LIBS:opto
-LIBS:atmel
-LIBS:contrib
-LIBS:valves
-LIBS:myLib
+EESchema Schematic File Version 4
 LIBS:proto-cache
-EELAYER 25 0
+EELAYER 26 0
 EELAYER END
 $Descr USLetter 8500 11000 portrait
@@
 $EndDescr
 $Comp
-L +5V #PWR0127
+L power:+5V #PWR0127
 U 1 1 56BE91DF
 P 3400 1400
@@
 $EndComp
 $Comp
-L +5V #PWR0128
+L power:+5V #PWR0128
 U 1 1 56BE91E5
 P 2800 1400
@@
 $EndComp
 $Comp
-L GND #PWR0129
+L power:GND #PWR0129
 U 1 1 56BE91EB
 P 2800 1500
@@
 $EndComp
 $Comp
-L GND #PWR0130
+L power:GND #PWR0130
 U 1 1 56BE91F1
 P 4350 1500
@@
 $EndComp
 $Comp
-L GND #PWR0131
+L power:GND #PWR0131
 U 1 1 56BE91F7
 P 3400 1500
@@
 $EndComp
 $Comp
-L GND #PWR0132
+L power:GND #PWR0132
 U 1 1 56BE91FD
 P 4950 1500
@@
 $EndComp
 $Comp
-L GND #PWR0133
+L power:GND #PWR0133
 U 1 1 56BE9203
 P 3400 2900
@@
 $EndComp
 $Comp
-L GND #PWR0134
+L power:GND #PWR0134
 U 1 1 56BE9209
 P 2800 2900
@@
 $EndComp
 $Comp
-L GND #PWR0135
+L power:GND #PWR0135
 U 1 1 56BE9215
 P 4350 3000
@@
 $EndComp
 $Comp
-L GND #PWR0136
+L power:GND #PWR0136
 U 1 1 56BE921B
 P 3400 4500
@@
 $EndComp
 $Comp
-L GND #PWR0137
+L power:GND #PWR0137
 U 1 1 56BE9227
 P 4350 4500
@@
 $EndComp
 $Comp
-L CONN_ZTEX_AB P1
+L myLib:CONN_ZTEX_AB P1
 U 1 1 56BE923A
 P 3050 2950
@@
 $EndComp
 $Comp
-L CONN_ZTEX_CD P2
+L myLib:CONN_ZTEX_CD P2
 U 1 1 56BE9241
 P 4600 2950
@@
 IPlatch_N
 $Comp
-L +12V #PWR0138
+L power:+12V #PWR0138
 U 1 1 56BE94C0
 P 5750 7150
@@
 $EndComp
 $Comp
-L +12V #PWR0139
+L power:+12V #PWR0139
 U 1 1 56BE94C6
 P 6350 7150
@@
 $EndComp
 $Comp
-L GND #PWR0140
+L power:GND #PWR0140
 U 1 1 56BE94CC
 P 5650 7650
@@
 $EndComp
 $Comp
-L GND #PWR0141
+L power:GND #PWR0141
 U 1 1 56BE94D2
 P 6450 7650
@@
 NoConn ~ 6300 6200
 Wire Wire Line
-	5650 7300 5650 7650
+	5650 7300 5650 7600
 Wire Wire Line
 	5650 7600 5800 7600
@@
 	6450 7600 6300 7600
 Wire Wire Line
-	6450 7300 6450 7650
+	6450 7300 6450 7600
 Wire Wire Line
 	6300 7300 6450 7300
 Wire Wire Line
-	6350 7150 6350 7500
+	6350 7150 6350 7400
 Wire Wire Line
 	6350 7400 6300 7400
@@
 	5800 7400 5750 7400
 Wire Wire Line
-	5750 7150 5750 7500
+	5750 7150 5750 7400
 Wire Wire Line
 	5750 7500 5800 7500
@@
 	3300 5550 3300 8300
 $Comp
-L CONN_02X16 P103
+L conn:CONN_02X16 P103
 U 1 1 56BF62BD
 P 1950 7000
@@
 $EndComp
 $Comp
-L MAX3033E U401
+L proto-rescue:MAX3033E U401
 U 1 1 56CCED40
 P 3950 6800
+AR Path="/56CCED40" Ref="U401"  Part="1"
+AR Path="/56BE8FCD/56CCED40" Ref="U401"  Part="1"
 F 0 "U401" H 4500 7050 60  0000 C CNN
 F 1 "MAX3033E" H 4050 7050 60  0000 C CNN
@@
 	3650 6800 3750 6800
 Wire Wire Line
-	3650 6600 3650 6800
+	3650 6600 3650 6700
 Wire Wire Line
 	3750 6700 3650 6700
 Connection ~ 3650 6700
 $Comp
-L +3V3 #PWR0142
+L power:+3V3 #PWR0142
 U 1 1 56CCF177
 P 3650 6600
@@
 $EndComp
 $Comp
-L CONN_02X04 P102
+L conn:CONN_02X04 P102
 U 1 1 56CCF1EB
 P 6050 7450
@@
 $EndComp
 $Comp
-L CONN_02X05 P101
+L conn:CONN_02X05 P101
 U 1 1 56CCF25D
 P 6050 6200
@@
 IPblank_N
 $Comp
-L GND #PWR0143
+L power:GND #PWR0143
 U 1 1 56CE3906
 P 4950 3000
@@
 $EndComp
 $Comp
-L GND #PWR0144
+L power:GND #PWR0144
 U 1 1 56CE3926
 P 4950 4500
@@
 RWTBT
 NoConn ~ 4350 1400
+Wire Wire Line
+	3650 6700 3650 6800
+Wire Wire Line
+	5750 7400 5750 7500
+Wire Wire Line
+	6350 7400 6350 7500
+Wire Wire Line
+	5650 7600 5650 7650
+Wire Wire Line
+	6450 7600 6450 7650
 $EndSCHEMATC
