File: board-qsic/io.sch (KiCad schematic (older format))
At the start: 36 parts, among them CON1 SD 0, CON2 SD 1, J601 USB_A, P2 Indicator Panel, U401 XC7A75T-CSG324, U601 MAX3033E, U602 USB3340

Commit message: Reworked board from template.  Changed schematic to let me use the bus drivers and level converters more efficiently so to get all the signals.
Parts:
- removed CON1: SD 0, myMods.pretty:microSD-3M-2900-series, symbol qsic-rescue:Micro_SD_Card_Det
- removed CON2: SD 1, myMods.pretty:microSD-3M-2900-series, symbol qsic-rescue:Micro_SD_Card_Det
- removed D601: LED 0, LEDs:LED-0603, symbol qsic-rescue:LED_Small
- removed D602: LED 1, LEDs:LED-0603, symbol qsic-rescue:LED_Small
- removed D603: LED 2, LEDs:LED-0603, symbol qsic-rescue:LED_Small
- removed D604: LED 3, LEDs:LED-0603, symbol qsic-rescue:LED_Small
- removed D605: LED 4, LEDs:LED-0603, symbol qsic-rescue:LED_Small
- removed D606: LED 5, LEDs:LED-0603, symbol qsic-rescue:LED_Small
- removed D607: LED 6, LEDs:LED-0603, symbol qsic-rescue:LED_Small
- removed D608: LED 7, LEDs:LED-0603, symbol qsic-rescue:LED_Small
- removed P2: Indicator Panel, Pin_Headers:Pin_Header_Angled_2x05, symbol qsic-rescue:CONN_02X05-conn
- removed R601, R602: 15k, Resistors_SMD:R_0603, symbol qsic-rescue:R-device
- removed R603, R604, R605, R606, R607, R608, R609, R610: R, Resistors_SMD:R_0603, symbol qsic-rescue:R-device
- removed R611, R612, R613, R614, R615, R616, R617, R619: 50k, Resistors_SMD:R_0603, symbol qsic-rescue:R-device
- removed R618, R620: 270k, Resistors_SMD:R_0603, symbol qsic-rescue:R-device
- removed U401: XC7A75T-CSG324, myMods.pretty:CSG324, symbol myLib:XC7A75T-CSG324
- removed U601: MAX3033E, Housings_SSOP:TSSOP-16_4.4x5mm_Pitch0.65mm, symbol myLib:MAX3033E
- removed U602: USB3340, Housings_DFN_QFN:QFN-32-1EP_5x5mm_Pitch0.5mm, symbol myLib:USB3340
- added C1301, C1303, C1304, C1309: 100nF, Capacitor_SMD:C_0603_1608Metric, symbol Device:C_Small
- added C1302: 150uF, Capacitor_SMD:CP_Elec_6.3x5.7, symbol Device:CP1_Small
- added C1305: 120uF, Capacitor_SMD:C_0603_1608Metric, symbol Device:C_Small
- added C1306, C1307: 1uF, Capacitor_SMD:C_0603_1608Metric, symbol Device:C_Small
- added C1308: 10nF, Capacitor_SMD:C_0603_1608Metric, symbol Device:C_Small
- added D1301, D1302, D1303, D1304, D1305, D1306, D1307, D1308: green, LED_SMD:LED_0603_1608Metric, symbol Device:LED_Small_ALT
- added P1301: Indicator Panel, myMods:Box_Header_2x05_P2.54mm, symbol Connector_Generic:Conn_02x05_Odd_Even
- added R1301, R1302, R1303, R1304, R1307, R1308, R1309, R1311: 240, Resistor_SMD:R_0603_1608Metric, symbol Device:R
- added R1305, R1306: 100k, Resistor_SMD:R_0603_1608Metric, symbol Device:R
- added R1310: 56.2k, Resistor_SMD:R_0603_1608Metric, symbol Device:R
- added R1312: 20k, Resistor_SMD:R_0603_1608Metric, symbol Device:R
- added R1313: 8.06k, Resistor_SMD:R_0603_1608Metric, symbol Device:R
- added U1301: TPS2561, Package_SON:VSON-10-1EP_3x3mm_P0.5mm_EP1.65x2.4mm_ThermalVias, symbol Interface_USB:TPS2561
- added U1302: USB3340, Package_DFN_QFN:QFN-32-1EP_5x5mm_P0.5mm_EP3.45x3.45mm, symbol myLib:USB3340
- added U1303: MAX3033E, Package_SO:TSSOP-16_4.4x5mm_P0.65mm, symbol myLib:MAX3033E
- added X1301: ASE-24.000MHz, Oscillator:Oscillator_SMD_Abracon_ASE-4Pin_3.2x2.5mm, symbol Oscillator:ASE-xxxMHz
- J1301: renamed from J601; footprint Connect:USB_A -> myMods:USB-A-Amphenol-UE27; symbol qsic-rescue:USB_A -> Connector:USB_A; manf# (none) -> UE27AC54100
- S1301: renamed from S601; footprint Buttons_Switches_ThroughHole:SW_DIP_x8_Slide -> Button_Switch_THT:SW_DIP_SPSTx08_Slide_6.7x21.88mm_W7.62mm_P2.54mm_LowProfile; manf# (none) -> 1825057-7
Connections:
- net labels added: 3V3, 5V, SW_0, SW_1, SW_2, SW_3, SW_4, SW_5, SW_6, SW_7, ip_blank, ip_clk, ip_data, ip_latch, usb0_clk60, usb0_d0, usb0_d1, usb0_d2, usb0_d3, usb0_d4, usb0_d5, usb0_d6, usb0_d7, usb0_dir, usb0_nxt, usb0_resetb, usb0_stp
- net labels removed: +3V3, +5V_USB, DIP_0, DIP_1, DIP_2, DIP_3, DIP_4, DIP_5, DIP_6, DIP_7, IPblank, IPclk, IPdata, IPlatch, SD0_CLK, SD0_DI, SD0_DO, SD0_NC1, SD0_NC2, SD0_~CS~/CD, SD1_CLK, SD1_DI, SD1_DO, SD1_NC1, SD1_NC2, SD1_~CS~/CD, USB_D+, USB_D-
- wire segments 120 -> 124
- no-connect marks 0 -> 5
Other:
- moved on the sheet: S1301
