File: board-qsic/qbus-interface.sch (KiCad schematic (older format))
At the start: 14 parts, among them J101 QBUS_A, J102 QBUS_B

Commit message: Design of prototype is done.  Needs checking before sending out.
Parts:
- added C601, C602, C603, C604, C605, C606, C607, C608, C609, C610, C611, C612, C613, C614, C615, C616, C617, C618, C619, C620, C621, C622, C623, C624, C625, C626, C627, C628, C629, C630, C631, C632, C633: 100nF, Capacitor_SMD:C_0603_1608Metric, symbol Device:C
- added U601, U602, U603, U604, U605, U606, U607, U608, U609, U610, U611: DS8641-small, Package_DIP:DIP-16_W7.62mm, symbol myLib:DS8641-small
- added U621, U622, U623, U624, U625, U626, U627, U628, U629, U630, U631: 74LVC8T245-small, Package_SO:SSOP-24_5.3x8.2mm_P0.65mm, symbol myLib:74LVC8T245-small
Connections:
- net 3V3: now also C623.1, C624.1, C625.1, C626.1, C627.1, C628.1, C629.1, C630.1, C631.1, C632.1, C633.1, U621.1 (VCCa), U622.1 (VCCa), U622.2 (A->B), U623.1 (VCCa), U624.1 (VCCa), U624.2 (A->B), U625.1 (VCCa), U626.1 (VCCa), U626.2 (A->B), U627.1 (VCCa), U628.1 (VCCa), U629.1 (VCCa), U629.2 (A->B), U630.1 (VCCa), U631.1 (VCCa), U631.2 (A->B)
- net 5V0: now also C601.1, C602.1, C603.1, C604.1, C605.1, C606.1, C607.1, C608.1, C609.1, C610.1, C611.1, C612.1, C613.1, C614.1, C615.1, C616.1, C617.1, C618.1, C619.1, C620.1, C621.1, C622.1, U601.16 (VCC), U602.16 (VCC), U603.16 (VCC), U604.16 (VCC), U605.16 (VCC), U606.16 (VCC), U607.16 (VCC), U608.16 (VCC), U609.16 (VCC), U610.16 (VCC), U611.16 (VCC), U621.23 (VCCb), U621.24 (VCCb), U622.23 (VCCb), U622.24 (VCCb), U623.23 (VCCb), U623.24 (VCCb), U624.23 (VCCb), U624.24 (VCCb), U625.23 (VCCb), U625.24 (VCCb), U626.23 (VCCb), U626.24 (VCCb), U627.23 (VCCb), U627.24 (VCCb), U628.23 (VCCb), U628.24 (VCCb), U629.23 (VCCb), U629.24 (VCCb), U630.23 (VCCb), U630.24 (VCCb), U631.23 (VCCb), U631.24 (VCCb)
- net BBS7: now also U604.4 (bus4)
- net BDAL0: now also U605.15 (bus1)
- net BDAL1: now also U606.1 (bus3)
- net BDAL10: now also U610.4 (bus4)
- net BDAL11: now also U610.15 (bus1)
- net BDAL12: now also U611.1 (bus3)
- net BDAL13: now also U611.4 (bus4)
- net BDAL14: now also U611.12 (bus2)
- net BDAL15: now also U611.15 (bus1)
- net BDAL16: now also U601.12 (bus2)
- net BDAL17: now also U601.15 (bus1)
- net BDAL18: now also U606.15 (bus1)
- net BDAL19: now also U607.1 (bus3)
- net BDAL2: now also U607.4 (bus4)
- net BDAL20: now also U607.12 (bus2)
- net BDAL21: now also U608.1 (bus3)
- net BDAL3: now also U607.15 (bus1)
- net BDAL4: now also U608.4 (bus4)
- net BDAL5: now also U608.12 (bus2)
- net BDAL6: now also U608.15 (bus1)
- net BDAL7: now also U609.1 (bus3)
- net BDAL8: now also U609.4 (bus4)
- net BDAL9: now also U609.12 (bus2)
- net BDCOK: now also U606.4 (bus4)
- net BDIN: now also U602.12 (bus2)
- net BDMGI: now also U605.1 (bus3)
- net BDMGO: now also U605.12 (bus2)
- net BDMR: now also U604.1 (bus3)
- net BDOUT: now also U602.1 (bus3)
- net BEVNT: now also U610.12 (bus2)
- net BHALT: now also U604.12 (bus2)
- net BIAKI: now also U603.15 (bus1)
- net BIAKO: now also U603.12 (bus2)
- net BINIT: now also U605.4 (bus4)
- net BIRQ4: now also U603.4 (bus4)
- net BIRQ5: now also U601.1 (bus3)
- net BIRQ6: now also U601.4 (bus4)
- net BIRQ7: now also U610.1 (bus3)
- net BPOK: now also U606.12 (bus2)
- net BREF: now also U604.15 (bus1)
- net BRPLY: now also U602.4 (bus4)
- net BSACK: now also U609.15 (bus1)
- net BSYNC: now also U602.15 (bus1)
- net BWTBT: now also U603.1 (bus3)
- net GND: now also C601.2, C602.2, C603.2, C604.2, C605.2, C606.2, C607.2, C608.2, C609.2, C610.2, C611.2, C612.2, C613.2, C614.2, C615.2, C616.2, C617.2, C618.2, C619.2, C620.2, C621.2, C622.2, C623.2, C624.2, C625.2, C626.2, C627.2, C628.2, C629.2, C630.2, C631.2, C632.2, C633.2, U601.7 (disB), U601.8 (GND), U601.9 (disA), U602.7 (disB), U602.8 (GND), U602.9 (disA), U603.14 (in1), U603.7 (disB), U603.8 (GND), U603.9 (disA), U604.11 (in2), U604.7 (disB), U604.8 (GND), U604.9 (disA), U605.2 (in3), U605.7 (disB), U605.8 (GND), U605.9 (disA), U606.11 (in2), U606.5 (in4), U606.7 (disB), U606.8 (GND), U606.9 (disA), U607.7 (disB), U607.8 (GND), U607.9 (disA), U608.7 (disB), U608.8 (GND), U608.9 (disA), U609.7 (disB), U609.8 (GND), U609.9 (disA), U610.11 (in2), U610.7 (disB), U610.8 (GND), U610.9 (disA), U611.7 (disB), U611.8 (GND), U611.9 (disA), U621.11 (GND), U621.12 (GND), U621.13 (GND), U621.2 (A->B), U621.22 (~OE), U622.11 (GND), U622.12 (GND), U622.13 (GND), U622.22 (~OE), U623.11 (GND), U623.12 (GND), U623.13 (GND), U623.2 (A->B), U623.22 (~OE), U624.11 (GND), U624.12 (GND), U624.13 (GND), U624.22 (~OE), U625.11 (GND), U625.12 (GND), U625.13 (GND), U625.2 (A->B), U625.22 (~OE), U626.11 (GND), U626.12 (GND), U626.13 (GND), U626.22 (~OE), U627.11 (GND), U627.12 (GND), U627.13 (GND), U627.2 (A->B), U627.22 (~OE), U628.11 (GND), U628.12 (GND), U628.13 (GND), U628.2 (A->B), U628.22 (~OE), U629.11 (GND), U629.12 (GND), U629.13 (GND), U629.22 (~OE), U630.11 (GND), U630.12 (GND), U630.13 (GND), U630.2 (A->B), U630.22 (~OE), U631.11 (GND), U631.12 (GND), U631.13 (GND), U631.22 (~OE)
- net RBS7: now also U623.7 (A)
- net RDAL0: now also U625.5 (A)
- net RDAL1: now also U625.10 (A)
- net RDAL10: now also U630.3 (A)
- net RDAL11: now also U630.5 (A)
- net RDAL12: now also U630.8 (A)
- net RDAL13: now also U630.7 (A)
- net RDAL14: now also U630.10 (A)
- net RDAL15: now also U630.9 (A)
- net RDAL16: now also U621.6 (A)
- net RDAL17: now also U621.5 (A)
- net RDAL18: now also U627.5 (A)
- net RDAL19: now also U627.8 (A)
- net RDAL2: now also U627.7 (A)
- net RDAL20: now also U627.10 (A)
- net RDAL21: now also U628.4 (A)
- net RDAL3: now also U627.9 (A)
- net RDAL4: now also U628.3 (A)
- net RDAL5: now also U628.6 (A)
- net RDAL6: now also U628.5 (A)
- net RDAL7: now also U628.8 (A)
- net RDAL8: now also U628.7 (A)
- net RDAL9: now also U628.10 (A)
- net RDCOK: now also U625.9 (A)
- net RDIN: now also U621.10 (A)
- net RDMGI: now also U625.4 (A)
- net RDMR: now also U623.8 (A)
- net RDOUT: now also U621.8 (A)
- net REVNT: now also U630.6 (A)
- net RHALT: now also U623.10 (A)
- net RIAKI: now also U623.5 (A)
- net RINIT: now also U625.3 (A)
- net RIRQ4: now also U623.3 (A)
- net RIRQ5: now also U621.4 (A)
- net RIRQ6: now also U621.3 (A)
- net RIRQ7: now also U630.4 (A)
- net RPOK: now also U627.6 (A)
- net RREF: now also U623.9 (A)
- net RRPLY: now also U621.7 (A)
- net RSACK: now also U628.9 (A)
- net RSYNC: now also U621.9 (A)
- net RWTBT: now also U623.4 (A)
- net TBS7: now also U624.7 (A)
- net TDAL0: now also U626.3 (A)
- net TDAL1: now also U626.5 (A)
- net TDAL10: now also U631.3 (A)
- net TDAL11: now also U631.5 (A)
- net TDAL12: now also U631.8 (A)
- net TDAL13: now also U631.7 (A)
- net TDAL14: now also U631.10 (A)
- net TDAL15: now also U631.9 (A)
- net TDAL16: now also U622.6 (A)
- net TDAL17: now also U622.5 (A)
- net TDAL18: now also U626.6 (A)
- net TDAL19: now also U626.8 (A)
- net TDAL2: now also U626.7 (A)
- net TDAL20: now also U626.10 (A)
- net TDAL21: now also U629.4 (A)
- net TDAL3: now also U626.9 (A)
- net TDAL4: now also U629.3 (A)
- net TDAL5: now also U629.6 (A)
- net TDAL6: now also U629.5 (A)
- net TDAL7: now also U629.8 (A)
- net TDAL8: now also U629.7 (A)
- net TDAL9: now also U629.10 (A)
- net TDIN: now also U622.10 (A)
- net TDMGO: now also U626.4 (A)
- net TDMR: now also U624.8 (A)
- net TDOUT: now also U622.8 (A)
- net TIAKO: now also U624.6 (A)
- net TINIT: now also U624.10 (A)
- net TIRQ4: now also U624.3 (A)
- net TIRQ5: now also U622.4 (A)
- net TIRQ6: now also U622.3 (A)
- net TIRQ7: now also U631.4 (A)
- net TREF: now also U624.9 (A)
- net TRPLY: now also U622.7 (A)
- net TSACK: now also U629.9 (A)
- net TSYNC: now also U622.9 (A)
- net TWTBT: now also U624.4 (A)
- new net: U605.14 (in1), U626.21 (B)
- new net: U605.13 (out1), U625.19 (B)
- new net: U606.2 (in3), U626.19 (B)
- new net: U606.3 (out3), U625.14 (B)
- new net: U607.5 (in4), U626.17 (B)
- new net: U607.6 (out4), U627.17 (B)
- new net: U607.14 (in1), U626.15 (B)
- new net: U607.13 (out1), U627.15 (B)
- new net: U608.5 (in4), U629.21 (B)
- new net: U608.6 (out4), U628.21 (B)
- new net: U608.11 (in2), U629.18 (B)
- new net: U608.10 (out2), U628.18 (B)
- new net: U608.14 (in1), U629.19 (B)
- new net: U608.13 (out1), U628.19 (B)
- new net: U609.2 (in3), U629.16 (B)
- new net: U609.3 (out3), U628.16 (B)
- new net: U609.5 (in4), U629.17 (B)
- new net: U609.6 (out4), U628.17 (B)
- new net: U609.11 (in2), U629.14 (B)
- new net: U609.10 (out2), U628.14 (B)
- new net: U610.5 (in4), U631.21 (B)
- new net: U610.6 (out4), U630.21 (B)
- new net: U610.14 (in1), U631.19 (B)
- new net: U610.13 (out1), U630.19 (B)
- new net: U611.2 (in3), U631.16 (B)
- new net: U611.3 (out3), U630.16 (B)
- new net: U611.5 (in4), U631.17 (B)
- new net: U611.6 (out4), U630.17 (B)
- new net: U611.11 (in2), U631.14 (B)
- new net: U611.10 (out2), U630.14 (B)
- new net: U611.14 (in1), U631.15 (B)
- new net: U611.13 (out1), U630.15 (B)
- new net: U601.11 (in2), U622.18 (B)
- new net: U601.10 (out2), U621.18 (B)
- new net: U601.14 (in1), U622.19 (B)
- new net: U601.13 (out1), U621.19 (B)
- new net: U606.14 (in1), U626.18 (B)
- new net: U606.13 (out1), U627.19 (B)
- new net: U607.2 (in3), U626.16 (B)
- new net: U607.3 (out3), U627.16 (B)
- new net: U607.11 (in2), U626.14 (B)
- new net: U607.10 (out2), U627.14 (B)
- new net: U608.2 (in3), U629.20 (B)
- new net: U608.3 (out3), U628.20 (B)
- new net: U604.5 (in4), U624.17 (B)
- new net: U604.6 (out4), U623.17 (B)
- new net: U603.2 (in3), U624.20 (B)
- new net: U603.3 (out3), U623.20 (B)
- new net: U602.14 (in1), U622.15 (B)
- new net: U602.13 (out1), U621.15 (B)
- new net: U602.11 (in2), U622.14 (B)
- new net: U602.10 (out2), U621.14 (B)
- new net: U602.2 (in3), U622.16 (B)
- new net: U602.3 (out3), U621.16 (B)
- new net: U602.5 (in4), U622.17 (B)
- new net: U602.6 (out4), U621.17 (B)
- new net: U604.14 (in1), U624.15 (B)
- new net: U604.13 (out1), U623.15 (B)
- new net: U603.5 (in4), U624.21 (B)
- new net: U603.6 (out4), U623.21 (B)
- new net: U601.2 (in3), U622.20 (B)
- new net: U601.3 (out3), U621.20 (B)
- new net: U601.5 (in4), U622.21 (B)
- new net: U601.6 (out4), U621.21 (B)
- new net: U610.2 (in3), U631.20 (B)
- new net: U610.3 (out3), U630.20 (B)
- new net: U604.2 (in3), U624.16 (B)
- new net: U604.3 (out3), U623.16 (B)
- new net: U609.14 (in1), U629.15 (B)
- new net: U609.13 (out1), U628.15 (B)
- new net: U605.5 (in4), U624.14 (B)
- new net: U605.6 (out4), U625.21 (B)
- new net: U604.10 (out2), U623.14 (B)
- new net: U606.6 (out4), U625.15 (B)
- new net: U606.10 (out2), U627.18 (B)
- new net: U610.10 (out2), U630.18 (B)
- new net: U603.13 (out1), U623.19 (B)
- new net: U603.11 (in2), U624.18 (B)
- new net: U605.3 (out3), U625.20 (B)
- new net: U605.11 (in2), U626.20 (B)
- no-connect marks 16 -> 18
Other:
- note added: "Receive Level Converters"
- note added: "Transmit Level Converters"
- moved on the sheet: J601, J602, R601, R602, R603, R604, R605, R606, R607, R608, RN606, RN607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
