File: board-qsic/qsic.sch (KiCad schematic (older format))
At the start: 2 parts, among them U401 XC7A75T-CSG324

Commit message: Reworked board from template.  Changed schematic to let me use the bus drivers and level converters more efficiently so to get all the signals.
Parts:
- removed B101: QBUS, myMods.pretty:Qbus-double, symbol myLib:QBUS
- removed U401: XC7A75T-CSG324, myMods.pretty:CSG324, symbol myLib:XC7A75T-CSG324
- added D101: LED_ALT, LED_SMD:LED_0603_1608Metric, symbol Device:LED_ALT
- added J101: Conn_02x05_Odd_Even, Connector:Tag-Connect_TC2050-IDC-FP_2x05_P1.27mm_Vertical, symbol Connector_Generic:Conn_02x05_Odd_Even
- added J102: Conn_02x07_Odd_Even, Connector_PinHeader_2.54mm:PinHeader_2x07_P2.54mm_Horizontal, symbol Connector_Generic:Conn_02x07_Odd_Even
- added LOGO101: Logo_Open_Hardware_Small, Symbol:KiCad-Logo2_5mm_SilkScreen, symbol Graphic:Logo_Open_Hardware_Small
- added R101: 240, Resistor_SMD:R_0603_1608Metric, symbol Device:R
- added R102, R103: 4.7k, Resistor_SMD:R_0603_1608Metric, symbol Device:R
- added U101: XC7A75T-CSG324, Package_BGA:BGA-324_15.0x15.0mm_Layout18x18_P0.8mm_Ball0.5mm_Pad0.4mm_NSMD, symbol FPGA_Xilinx_Artix7:XC7A75T-CSG324
Connections:
- net labels added: 1V0, 1V5, 1V8, 3V3, 5V0, TCK, TDI, TDO, TMS
- net labels removed: +5V, BDAL0, BDAL1, BDAL10, BDAL11, BDAL12, BDAL13, BDAL14, BDAL15, BDAL16, BDAL17, BDAL18, BDAL19, BDAL2, BDAL20, BDAL21, BDAL3, BDAL4, BDAL5, BDAL6, BDAL7, BDAL8, BDAL9, BDAL[0..21], RBS7, RDAL[0..21], RDCOK, RDIN, RDMGI, RDMR, RDOUT, REVNT, RHALT, RIAKI, RINIT, RIRQ4, RIRQ5, RIRQ6, RIRQ7, RPOK, RREF, RRPLY, RSACK, RSYNC, RWTBT, TBS7, TDAL[0..21], TDIN, TDMGO, TDMR, TDOUT, TIAKO, TINIT, TIRQ4, TIRQ5, TIRQ6, TIRQ7, TREF, TRPLY, TSACK, TSYNC, TWTBT
- wire segments 74 -> 38
- no-connect marks 15 -> 3
Other:
- note added: "QSIC - QBUS Storage & I/O Card"
- note removed: "QSIC - QBUS Storage I/O Card"

Commit message: Design of prototype is done.  Needs checking before sending out.
Parts:
- D101: value LED_ALT -> green; manf# (none) -> LTST-C190KGKT
- J101, LOGO101: DNP (none) -> x
- J102: footprint Connector_PinHeader_2.54mm:PinHeader_2x07_P2.54mm_Horizontal -> Connector_PinHeader_2.00mm:PinHeader_2x07_P2.00mm_Vertical; DNP (none) -> x
Connections:
- net 3V3: now also J101.1 (Pin_1), J102.2 (Pin_2), U101.P8 (CFGBVS_0)
- net GND: now also U101.J10 (VP_0), U101.K9 (VN_0), U101.L10 (DXP_0), U101.L9 (DXN_0); no longer J101.1 (Pin_1)
- net QBUS/CCLK renamed QBUS & I/O/CCLK
Changed lines of the file:
@@
 $Descr A 11000 8500
 encoding utf-8
-Sheet 1 53
+Sheet 1 5
 Title "QSIC - QBUS Storage & I/O Card"
-Date "2019-09-30"
+Date "2019-10-07"
 Rev "0.2"
 Comp "QSIC - QBUS Storage & I/O Card"
@@
 $EndComp
 $Sheet
-S 9000 4800 650  700
-U 5D8E0230
-F0 "SD 0" 60
-F1 "sd.sch" 60
-F2 "DAT2" B R 9650 5100 60
-F3 "DAT3" B R 9650 5200 60
-F4 "CMD" I L 9000 5200 60
-F5 "CLK" I L 9000 5100 60
-F6 "DAT0" B R 9650 4900 60
-F7 "DAT1" B R 9650 5000 60
-F8 "DET" O R 9650 5400 60
-F9 "3V3" I L 9000 4900 60
-$EndSheet
-$Sheet
 S 9000 4025 650  550
 U 5D8F7A71
@@
 $EndSheet
 $Sheet
-S 9000 5750 650  700
-U 5D933A84
-F0 "SD 1" 60
-F1 "sd.sch" 60
-F2 "DAT2" B R 9650 6050 60
-F3 "DAT3" B R 9650 6150 60
-F4 "CMD" I L 9000 6150 60
-F5 "CLK" I L 9000 6050 60
-F6 "DAT0" B R 9650 5850 60
-F7 "DAT1" B R 9650 5950 60
-F8 "DET" O R 9650 6350 60
-F9 "3V3" I L 9000 5850 60
-$EndSheet
-$Sheet
 S 7000 1975 625  575
 U 5DCB8CA6
-F0 "QBUS" 60
+F0 "QBUS & I/O" 60
 F1 "qbus.sch" 60
 F2 "3V3" I L 7000 2075 60
 F3 "5V0" O R 7625 2075 60
 F4 "CCLK" I L 7000 2300 60
+F5 "1V8" I L 7000 2175 60
 $EndSheet
 Text Notes 8850 1200 2    250  ~ 50
 QSIC - QBUS Storage & I/O Card
-$Sheet
-S 7575 3600 675  625
-U 5DA36495
-F0 "IO" 60
-F1 "io.sch" 60
-$EndSheet
 $Sheet
 S 8225 1975 550  525
@@
 P 4925 4375
 F 0 "D101" H 4918 4591 50  0000 C CNN
-F 1 "LED_ALT" H 4918 4500 50  0000 C CNN
+F 1 "green" H 4918 4500 50  0000 C CNN
 F 2 "LED_SMD:LED_0603_1608Metric" H 4925 4375 50  0001 C CNN
 F 3 "~" H 4925 4375 50  0001 C CNN
+F 4 "LTST-C190KGKT" H 4925 4375 50  0001 C CNN "manf#"
 	1    4925 4375
 	1    0    0    -1
@@
 L power:GND #PWR0210
 U 1 1 5DAA622F
-P 4525 5400
-F 0 "#PWR0210" H 4525 5150 50  0001 C CNN
-F 1 "GND" H 4530 5227 50  0001 C CNN
-F 2 "" H 4525 5400 50  0001 C CNN
-F 3 "" H 4525 5400 50  0001 C CNN
-	1    4525 5400
+P 4525 5725
+F 0 "#PWR0210" H 4525 5475 50  0001 C CNN
+F 1 "GND" H 4530 5552 50  0001 C CNN
+F 2 "" H 4525 5725 50  0001 C CNN
+F 3 "" H 4525 5725 50  0001 C CNN
+	1    4525 5725
 	1    0    0    -1
 $EndComp
@@
 	4425 5375 4525 5375
 Connection ~ 4525 5375
-Wire Wire Line
-	4525 5375 4525 5400
 Wire Wire Line
 	4425 3875 5975 3875
@@
 F 2 "Connector:Tag-Connect_TC2050-IDC-FP_2x05_P1.27mm_Vertical" H 2525 6675 50  0001 C CNN
 F 3 "~" H 2525 6675 50  0001 C CNN
+F 4 "x" H 2525 6675 50  0001 C CNN "DNP"
 	1    2525 6675
 	1    0    0    -1
@@
 F 0 "J102" H 3700 7217 50  0000 C CNN
 F 1 "Conn_02x07_Odd_Even" H 3700 7126 50  0000 C CNN
-F 2 "Connector_PinHeader_2.54mm:PinHeader_2x07_P2.54mm_Horizontal" H 3650 6700 50  0001 C CNN
+F 2 "Connector_PinHeader_2.00mm:PinHeader_2x07_P2.00mm_Vertical" H 3650 6700 50  0001 C CNN
 F 3 "~" H 3650 6700 50  0001 C CNN
+F 4 "x" H 3650 6700 50  0001 C CNN "DNP"
 	1    3650 6700
 	1    0    0    -1
@@
 Wire Wire Line
 	2325 6925 2325 6875
-Connection ~ 2325 6575
-Wire Wire Line
-	2325 6575 2325 6475
 Connection ~ 2325 6675
 Wire Wire Line
@@
 F 2 "Symbol:KiCad-Logo2_5mm_SilkScreen" H 1450 6725 50  0001 C CNN
 F 3 "~" H 1450 6725 50  0001 C CNN
+F 4 "x" H 1450 6725 50  0001 C CNN "DNP"
 	1    1450 6725
 	1    0    0    -1
 $EndComp
+Text Label 3950 6400 0    60   ~ 0
+3V3
+Text Label 2325 6475 2    60   ~ 0
+3V3
+Text Label 9000 4125 2    60   ~ 0
+1V5
+Text Label 7000 2175 2    60   ~ 0
+1V8
+Wire Wire Line
+	4425 4975 4525 4975
+Wire Wire Line
+	4525 4975 4525 5075
+Wire Wire Line
+	4425 5075 4525 5075
+Connection ~ 4525 5075
+Wire Wire Line
+	4525 5075 4525 5275
+Wire Wire Line
+	4425 5575 4525 5575
+Wire Wire Line
+	4525 5575 4525 5675
+Wire Wire Line
+	4425 5675 4525 5675
+Connection ~ 4525 5675
+Wire Wire Line
+	4525 5675 4525 5725
+Wire Wire Line
+	4525 5375 4525 5575
+Connection ~ 4525 5575
+Connection ~ 4525 5275
+Text Label 4425 4775 0    60   ~ 0
+3V3
 $EndSCHEMATC

Commit message: Added fiducials
Parts:
- added FID101, FID102, FID103, FID104, FID105: Fiducial, Fiducial:Fiducial_1mm_Mask2mm, symbol Mechanical:Fiducial
- added R104, R105: 10k, Resistor_SMD:R_0603_1608Metric, symbol Device:R
Connections:
- net 3V3: now also R104.1, R105.1
- net TCK: now also R105.2
- net TMS: now also R104.2
Changed lines of the file:
@@
 Text Label 4425 4775 0    60   ~ 0
 3V3
+$Comp
+L Device:R R?
+U 1 1 5DB4FA0E
+P 4775 3100
+AR Path="/5DCB8CA6/5DB4FA0E" Ref="R?"  Part="1"
+AR Path="/5DB4FA0E" Ref="R104"  Part="1"
+F 0 "R104" H 4845 3146 50  0000 L CNN
+F 1 "10k" H 4845 3055 50  0000 L CNN
+F 2 "Resistor_SMD:R_0603_1608Metric" V 4705 3100 50  0001 C CNN
+F 3 "~" H 4775 3100 50  0001 C CNN
+	1    4775 3100
+	1    0    0    -1
+$EndComp
+$Comp
+L Device:R R?
+U 1 1 5DB5007F
+P 5100 3100
+AR Path="/5DCB8CA6/5DB5007F" Ref="R?"  Part="1"
+AR Path="/5DB5007F" Ref="R105"  Part="1"
+F 0 "R105" H 5170 3146 50  0000 L CNN
+F 1 "10k" H 5170 3055 50  0000 L CNN
+F 2 "Resistor_SMD:R_0603_1608Metric" V 5030 3100 50  0001 C CNN
+F 3 "~" H 5100 3100 50  0001 C CNN
+	1    5100 3100
+	1    0    0    -1
+$EndComp
+Wire Wire Line
+	4425 3575 4775 3575
+Wire Wire Line
+	4775 3575 4775 3250
+Wire Wire Line
+	4425 3675 5100 3675
+Wire Wire Line
+	5100 3675 5100 3250
+Text Label 4700 2900 2    60   ~ 0
+3V3
+Wire Wire Line
+	4700 2900 4775 2900
+Wire Wire Line
+	5100 2900 5100 2950
+Wire Wire Line
+	4775 2950 4775 2900
+Connection ~ 4775 2900
+Wire Wire Line
+	4775 2900 5100 2900
+$Comp
+L Mechanical:Fiducial FID101
+U 1 1 5DBEFBB8
+P 5675 6900
+F 0 "FID101" H 5760 6946 50  0000 L CNN
+F 1 "Fiducial" H 5760 6855 50  0000 L CNN
+F 2 "Fiducial:Fiducial_1mm_Mask2mm" H 5675 6900 50  0001 C CNN
+F 3 "~" H 5675 6900 50  0001 C CNN
+	1    5675 6900
+	1    0    0    -1
+$EndComp
+$Comp
+L Mechanical:Fiducial FID102
+U 1 1 5DBF958E
+P 5675 7125
+F 0 "FID102" H 5760 7171 50  0000 L CNN
+F 1 "Fiducial" H 5760 7080 50  0000 L CNN
+F 2 "Fiducial:Fiducial_1mm_Mask2mm" H 5675 7125 50  0001 C CNN
+F 3 "~" H 5675 7125 50  0001 C CNN
+	1    5675 7125
+	1    0    0    -1
+$EndComp
+$Comp
+L Mechanical:Fiducial FID103
+U 1 1 5DBF9A00
+P 5675 7350
+F 0 "FID103" H 5760 7396 50  0000 L CNN
+F 1 "Fiducial" H 5760 7305 50  0000 L CNN
+F 2 "Fiducial:Fiducial_1mm_Mask2mm" H 5675 7350 50  0001 C CNN
+F 3 "~" H 5675 7350 50  0001 C CNN
+	1    5675 7350
+	1    0    0    -1
+$EndComp
+$Comp
+L Mechanical:Fiducial FID104
+U 1 1 5DBF9E8E
+P 5675 7575
+F 0 "FID104" H 5760 7621 50  0000 L CNN
+F 1 "Fiducial" H 5760 7530 50  0000 L CNN
+F 2 "Fiducial:Fiducial_1mm_Mask2mm" H 5675 7575 50  0001 C CNN
+F 3 "~" H 5675 7575 50  0001 C CNN
+	1    5675 7575
+	1    0    0    -1
+$EndComp
+$Comp
+L Mechanical:Fiducial FID105
+U 1 1 5DBFCFB6
+P 5675 7800
+F 0 "FID105" H 5760 7846 50  0000 L CNN
+F 1 "Fiducial" H 5760 7755 50  0000 L CNN
+F 2 "Fiducial:Fiducial_1mm_Mask2mm" H 5675 7800 50  0001 C CNN
+F 3 "~" H 5675 7800 50  0001 C CNN
+	1    5675 7800
+	1    0    0    -1
+$EndComp
 $EndSCHEMATC
