File: board-wirewrap/proto.sch (KiCad schematic (older format))
At the start: 54 parts, among them CON101 Micro_SD_Card, P1 AB, P101 Data, P102 Power, P103 DIL8, P2 CD, SW101 RESET, U1 DS8641-LR, U101 Am2908, U102 Am2908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

Commit message: Annotated all the components so the netlist works right.
Parts:
- gave numbers to parts that had none: 8

Commit message: Update to KiCad v5
Parts:
- B101: symbol QBUS -> proto-rescue:QBUS
- C101, C102: symbol CP1_Small -> proto-rescue:CP1_Small
- CON101: symbol Micro_SD_Card -> proto-rescue:Micro_SD_Card
- D101, D102, D103, D104: symbol Led_Small -> proto-rescue:Led_Small
- P1: symbol CONN_ZTEX_AB -> proto-rescue:CONN_ZTEX_AB
- P101: symbol CONN_02X04 -> proto-rescue:CONN_02X04
- P102: symbol CONN_02X05 -> proto-rescue:CONN_02X05
- P103: symbol DIL8 -> proto-rescue:DIL8
- P2: symbol CONN_ZTEX_CD -> proto-rescue:CONN_ZTEX_CD
- R101, R102, R103, R104, R105, R106, R107, R108, R109, R110, R111, R112, R113, R114, R115, R116, R117: symbol R -> proto-rescue:R
- SW101: symbol SW_PUSH_SMALL -> proto-rescue:SW_PUSH_SMALL
- U1, U2, U3, U4, U5: symbol DS8641-LR -> proto-rescue:DS8641-LR
- U101, U102, U103, U104, U105, U106: symbol Am2908 -> proto-rescue:Am2908
- U107, U108, U109, U115, U116, U117, U118, U119: symbol 74LVC7T245 -> proto-rescue:74LVC7T245
- U110, U111, U112: symbol MAX3488 -> proto-rescue:MAX3488
- U120: symbol LT1129MPST-3.3 -> proto-rescue:LT1129MPST-3.3
