File: board-smt/bus-dal.sch (KiCad schematic (older format))
At the start: 94 parts, among them Q201 Dual_NMOS, Q202 Dual_NMOS, Q203 Dual_NMOS, Q204 Dual_NMOS, Q205 Dual_NMOS, Q206 Dual_NMOS, Q207 Dual_NMOS, Q208 Dual_NMOS, Q209 Dual_NMOS, Q210 Dual_NMOS, Q211 Dual_NMOS, Q212 Dual_NMOS, U201 CMP401, U202 CMP401, U203 CMP401, U204 CMP401, U205 CMP401, U206 CMP401, U301 CMP401, U303 CMP401, U304 CMP401, U305 CMP401

Commit message: Moved comparator power connections to separate symbols.
Connections:
- net labels added: +1V5_ref
- net labels removed: +1V5, +3V3, +5V
- wire segments 336 -> 215

Commit message: Updated to KiCad v5
Parts:
- Q201, Q202, Q203, Q204, Q205, Q206, Q207, Q208, Q209, Q210, Q211, Q212: symbol Dual_NMOS -> myLib:Dual_NMOS
- R201, R202, R203, R204, R205, R206, R207, R208, R209, R210, R211, R212, R213, R214, R215, R216, R217, R218, R219, R220, R221, R222, R223, R224, R225, R226, R227, R228, R229, R230, R231, R232, R233, R234, R235, R236, R237, R238, R239, R240, R241, R242, R243, R244, R245, R246, R247, R248, R249, R250, R251, R252, R253, R254, R255, R256, R257, R258, R259, R260, R261, R262, R263, R264, R265, R266, R267, R268, R269, R270, R271, R272: symbol R -> device:R
- U201, U202, U203, U204, U205, U206, U301, U303, U304, U305: symbol CMP401 -> myLib:CMP401
Connections:
- wire segments 215 -> 286

Commit message: Updated to KiCad v5
Parts:
- R201, R202, R203, R204, R205, R206, R207, R208, R209, R210, R211, R212, R213, R214, R215, R216, R217, R218, R219, R220, R221, R222, R223, R224, R225, R226, R227, R228, R229, R230, R231, R232, R233, R234, R235, R236, R237, R238, R239, R240, R241, R242, R243, R244, R245, R246, R247, R248, R249, R250, R251, R252, R253, R254, R255, R256, R257, R258, R259, R260, R261, R262, R263, R264, R265, R266, R267, R268, R269, R270, R271, R272: symbol device:R -> qsic-rescue:R-device

Commit message: These are all old changes in directories that are now historical.
Parts:
- R201, R202, R203, R204, R205, R206, R207, R208, R209, R210, R211, R212, R213, R214, R215, R216, R217, R218, R219, R220, R221, R222, R223, R224, R225, R226, R227, R228, R229, R230, R231, R232, R233, R234, R235, R236, R237, R238, R239, R240, R241, R242, R243, R244, R245, R246, R247, R248, R249, R250, R251, R252, R253, R254, R255, R256, R257, R258, R259, R260, R261, R262, R263, R264, R265, R266, R267, R268, R269, R270, R271, R272: footprint Resistors_SMD:R_0603 -> Resistor_SMD:R_0603_1608Metric
