File: board-smt/io.sch (KiCad schematic (older format))
At the start: 35 parts, among them CON1 SD 0, CON2 SD 1, P1 USB_A, P2 Indicator Panel, U401 XC7A75T-CSG324, U601 MAX3033E

Commit message: Moved comparator power connections to separate symbols.
Parts:
- removed P1: USB_A, Connect:USB_A, symbol USB_A
- added J601: USB_A, symbol USB_A
Connections:
- wire segments 82 -> 81
Changed lines of the file:
@@
 EESchema Schematic File Version 2
+LIBS:qsic-rescue
 LIBS:power
 LIBS:device
@@
 Sheet 6 6
 Title "I/O Ports"
-Date "2017-03-12"
+Date "2017-10-31"
 Rev "0.1"
 Comp "Vintage Computer Engineering"
@@
 $EndComp
 $Comp
-L USB_A P1
-U 1 1 58C5DD20
-P 5850 6100
-F 0 "P1" H 6050 5900 50  0000 C CNN
-F 1 "USB_A" H 5800 6300 50  0000 C CNN
-F 2 "Connect:USB_A" V 5800 6000 50  0001 C CNN
-F 3 "" V 5800 6000 50  0000 C CNN
-	1    5850 6100
-	0    1    1    0
-$EndComp
-$Comp
 L CONN_02X05 P2
 U 1 1 58C5E53F
@@
 $EndComp
 $Comp
-L GND #PWR0221
+L GND #PWR0181
 U 1 1 58C7C181
 P 8000 2300
-F 0 "#PWR0221" H 8000 2050 50  0001 C CNN
+F 0 "#PWR0181" H 8000 2050 50  0001 C CNN
 F 1 "GND" H 8000 2150 50  0001 C CNN
 F 2 "" H 8000 2300 50  0000 C CNN
@@
 	8000 2300 8000 2250
 $Comp
-L GND #PWR0222
+L GND #PWR0182
 U 1 1 58C7C5A9
 P 8200 2000
-F 0 "#PWR0222" H 8200 1750 50  0001 C CNN
+F 0 "#PWR0182" H 8200 1750 50  0001 C CNN
 F 1 "GND" H 8200 1850 50  0001 C CNN
 F 2 "" H 8200 2000 50  0000 C CNN
@@
 	8200 1700 8200 2000
 $Comp
-L +3V3 #PWR0223
+L +3V3 #PWR0183
 U 1 1 58C7C6E8
 P 8200 750
-F 0 "#PWR0223" H 8200 600 50  0001 C CNN
+F 0 "#PWR0183" H 8200 600 50  0001 C CNN
 F 1 "+3V3" H 8200 890 50  0000 C CNN
 F 2 "" H 8200 750 50  0000 C CNN
@@
 $EndComp
 $Comp
-L GND #PWR0224
+L GND #PWR0184
 U 1 1 58C7CFA0
 P 8000 4050
-F 0 "#PWR0224" H 8000 3800 50  0001 C CNN
+F 0 "#PWR0184" H 8000 3800 50  0001 C CNN
 F 1 "GND" H 8000 3900 50  0001 C CNN
 F 2 "" H 8000 4050 50  0000 C CNN
@@
 	8000 4050 8000 4000
 $Comp
-L GND #PWR0225
+L GND #PWR0185
 U 1 1 58C7CFC2
 P 8200 3750
-F 0 "#PWR0225" H 8200 3500 50  0001 C CNN
+F 0 "#PWR0185" H 8200 3500 50  0001 C CNN
 F 1 "GND" H 8200 3600 50  0001 C CNN
 F 2 "" H 8200 3750 50  0000 C CNN
@@
 	8200 3450 8200 3750
 $Comp
-L +3V3 #PWR0226
+L +3V3 #PWR0186
 U 1 1 58C7CFCA
 P 8200 2500
-F 0 "#PWR0226" H 8200 2350 50  0001 C CNN
+F 0 "#PWR0186" H 8200 2350 50  0001 C CNN
 F 1 "+3V3" H 8200 2640 50  0000 C CNN
 F 2 "" H 8200 2500 50  0000 C CNN
@@
 Connection ~ 8000 2550
 $Comp
-L GND #PWR0227
+L GND #PWR0187
 U 1 1 58C7DAE3
 P 10000 2200
-F 0 "#PWR0227" H 10000 1950 50  0001 C CNN
+F 0 "#PWR0187" H 10000 1950 50  0001 C CNN
 F 1 "GND" H 10000 2050 50  0001 C CNN
 F 2 "" H 10000 2200 50  0000 C CNN
@@
 $EndComp
 $Comp
-L GND #PWR0228
+L GND #PWR0188
 U 1 1 58C7DB1B
 P 10000 3950
-F 0 "#PWR0228" H 10000 3700 50  0001 C CNN
+F 0 "#PWR0188" H 10000 3700 50  0001 C CNN
 F 1 "GND" H 10000 3800 50  0001 C CNN
 F 2 "" H 10000 3950 50  0000 C CNN
@@
 	10000 2200 10000 2100
 $Comp
-L GND #PWR0229
+L GND #PWR0189
 U 1 1 58C7DE50
 P 5950 6450
-F 0 "#PWR0229" H 5950 6200 50  0001 C CNN
+F 0 "#PWR0189" H 5950 6200 50  0001 C CNN
 F 1 "GND" H 5950 6300 50  0001 C CNN
 F 2 "" H 5950 6450 50  0000 C CNN
@@
 Wire Wire Line
 	5950 6450 5950 6400
-$Comp
-L GND #PWR0230
-U 1 1 58C7DED7
-P 5500 6450
-F 0 "#PWR0230" H 5500 6200 50  0001 C CNN
-F 1 "GND" H 5500 6300 50  0001 C CNN
-F 2 "" H 5500 6450 50  0000 C CNN
-F 3 "" H 5500 6450 50  0000 C CNN
-	1    5500 6450
-	1    0    0    -1
-$EndComp
-Wire Wire Line
-	5550 6200 5500 6200
-Wire Wire Line
-	5500 6200 5500 6450
-Wire Wire Line
-	5500 5850 5500 5900
-Wire Wire Line
-	5500 5900 5550 5900
-$Comp
-L +5V_USB #PWR0231
+Wire Wire Line
+	5950 6400 5850 6400
+Wire Wire Line
+	5500 5700 5500 5800
+Wire Wire Line
+	5500 5800 5550 5800
+$Comp
+L +5V_USB #PWR0190
 U 1 1 58C7E0AF
-P 5500 5850
-F 0 "#PWR0231" H 5500 5700 50  0001 C CNN
-F 1 "+5V_USB" H 5500 5990 50  0000 C CNN
-F 2 "" H 5500 5850 50  0000 C CNN
-F 3 "" H 5500 5850 50  0000 C CNN
-	1    5500 5850
-	1    0    0    -1
-$EndComp
+P 5500 5700
+F 0 "#PWR0190" H 5500 5550 50  0001 C CNN
+F 1 "+5V_USB" H 5500 5840 50  0000 C CNN
+F 2 "" H 5500 5700 50  0000 C CNN
+F 3 "" H 5500 5700 50  0000 C CNN
+	1    5500 5700
+	1    0    0    -1
+$EndComp
+Text Label 4850 6100 2    60   ~ 0
+USB_D-
 Text Label 4850 6000 2    60   ~ 0
-USB_D-
-Text Label 4850 6100 2    60   ~ 0
 USB_D+
 $Comp
@@
 $EndComp
 $Comp
-L +3V3 #PWR0232
+L +3V3 #PWR0191
 U 1 1 58C6D13C
 P 6950 4500
-F 0 "#PWR0232" H 6950 4350 50  0001 C CNN
+F 0 "#PWR0191" H 6950 4350 50  0001 C CNN
 F 1 "+3V3" H 6950 4640 50  0000 C CNN
 F 2 "" H 6950 4500 50  0000 C CNN
@@
 Connection ~ 5100 6100
 $Comp
-L GND #PWR0233
+L GND #PWR0192
 U 1 1 58C6CBD5
 P 5300 6450
-F 0 "#PWR0233" H 5300 6200 50  0001 C CNN
+F 0 "#PWR0192" H 5300 6200 50  0001 C CNN
 F 1 "GND" H 5300 6300 50  0001 C CNN
 F 2 "" H 5300 6450 50  0000 C CNN
@@
 $EndComp
 $Comp
-L GND #PWR0234
+L GND #PWR0193
 U 1 1 58C6CC16
 P 5100 6450
-F 0 "#PWR0234" H 5100 6200 50  0001 C CNN
+F 0 "#PWR0193" H 5100 6200 50  0001 C CNN
 F 1 "GND" H 5100 6300 50  0001 C CNN
 F 2 "" H 5100 6450 50  0000 C CNN
@@
 DIP_7
 $Comp
-L GND #PWR0235
+L GND #PWR0194
 U 1 1 58C72C63
 P 5950 3950
-F 0 "#PWR0235" H 5950 3700 50  0001 C CNN
+F 0 "#PWR0194" H 5950 3700 50  0001 C CNN
 F 1 "GND" H 5950 3800 50  0001 C CNN
 F 2 "" H 5950 3950 50  0000 C CNN
@@
 U 1 1 58C73DB2
 P 5350 900
-F 0 "D601" H 5300 1025 50  0000 L CNN
-F 1 "LED 0" H 5450 1000 50  0000 L CNN
+F 0 "D601" H 5200 1000 50  0000 L CNN
+F 1 "LED 0" H 5400 950 50  0000 L CNN
 F 2 "LEDs:LED-0603" V 5350 900 50  0001 C CNN
 F 3 "" V 5350 900 50  0000 C CNN
@@
 U 1 1 58C73F83
 P 5350 1150
-F 0 "D602" H 5300 1275 50  0000 L CNN
-F 1 "LED 1" H 5450 1250 50  0000 L CNN
+F 0 "D602" H 5200 1250 50  0000 L CNN
+F 1 "LED 1" H 5400 1200 50  0000 L CNN
 F 2 "LEDs:LED-0603" V 5350 1150 50  0001 C CNN
 F 3 "" V 5350 1150 50  0000 C CNN
@@
 U 1 1 58C741C5
 P 5350 1400
-F 0 "D603" H 5300 1525 50  0000 L CNN
-F 1 "LED 2" H 5450 1500 50  0000 L CNN
+F 0 "D603" H 5200 1500 50  0000 L CNN
+F 1 "LED 2" H 5400 1450 50  0000 L CNN
 F 2 "LEDs:LED-0603" V 5350 1400 50  0001 C CNN
 F 3 "" V 5350 1400 50  0000 C CNN
@@
 U 1 1 58C741CC
 P 5350 1650
-F 0 "D604" H 5300 1775 50  0000 L CNN
-F 1 "LED 3" H 5450 1750 50  0000 L CNN
+F 0 "D604" H 5200 1750 50  0000 L CNN
+F 1 "LED 3" H 5400 1700 50  0000 L CNN
 F 2 "LEDs:LED-0603" V 5350 1650 50  0001 C CNN
 F 3 "" V 5350 1650 50  0000 C CNN
@@
 U 1 1 58C744B9
 P 5350 1900
-F 0 "D605" H 5300 2025 50  0000 L CNN
-F 1 "LED 4" H 5450 2000 50  0000 L CNN
+F 0 "D605" H 5200 2000 50  0000 L CNN
+F 1 "LED 4" H 5400 1950 50  0000 L CNN
 F 2 "LEDs:LED-0603" V 5350 1900 50  0001 C CNN
 F 3 "" V 5350 1900 50  0000 C CNN
@@
 U 1 1 58C744C0
 P 5350 2150
-F 0 "D606" H 5300 2275 50  0000 L CNN
-F 1 "LED 5" H 5450 2250 50  0000 L CNN
+F 0 "D606" H 5200 2250 50  0000 L CNN
+F 1 "LED 5" H 5400 2200 50  0000 L CNN
 F 2 "LEDs:LED-0603" V 5350 2150 50  0001 C CNN
 F 3 "" V 5350 2150 50  0000 C CNN
@@
 U 1 1 58C744C7
 P 5350 2400
-F 0 "D607" H 5300 2525 50  0000 L CNN
-F 1 "LED 6" H 5450 2500 50  0000 L CNN
+F 0 "D607" H 5200 2500 50  0000 L CNN
+F 1 "LED 6" H 5400 2450 50  0000 L CNN
 F 2 "LEDs:LED-0603" V 5350 2400 50  0001 C CNN
 F 3 "" V 5350 2400 50  0000 C CNN
@@
 U 1 1 58C744CE
 P 5350 2650
-F 0 "D608" H 5300 2775 50  0000 L CNN
-F 1 "LED 7" H 5450 2750 50  0000 L CNN
+F 0 "D608" H 5200 2750 50  0000 L CNN
+F 1 "LED 7" H 5400 2700 50  0000 L CNN
 F 2 "LEDs:LED-0603" V 5350 2650 50  0001 C CNN
 F 3 "" V 5350 2650 50  0000 C CNN
@@
 $EndComp
 $Comp
-L +3V3 #PWR0236
+L +3V3 #PWR0195
 U 1 1 58C74D20
 P 6100 800
-F 0 "#PWR0236" H 6100 650 50  0001 C CNN
+F 0 "#PWR0195" H 6100 650 50  0001 C CNN
 F 1 "+3V3" H 6100 940 50  0000 C CNN
 F 2 "" H 6100 800 50  0000 C CNN
@@
 	5950 2400 6100 2400
 Wire Wire Line
-	5950 2650 6100 2650
-Wire Wire Line
-	6100 2650 6100 800
+	6100 2650 5950 2650
+Wire Wire Line
+	6100 800  6100 2650
 Connection ~ 6100 900
 Connection ~ 6100 1150
@@
 Text Label 5250 2650 2    60   ~ 0
 LED_7
+$Comp
+L USB_A J601
+U 1 1 59C838C8
+P 5850 6000
+F 0 "J601" H 5650 6450 50  0000 L CNN
+F 1 "USB_A" H 5650 6350 50  0000 L CNN
+F 2 "" H 6000 5950 50  0001 C CNN
+F 3 "" H 6000 5950 50  0001 C CNN
+	1    5850 6000
+	-1   0    0    -1
+$EndComp
 $EndSCHEMATC

Commit message: Little fixups
Parts:
- P2: footprint Socket_Strips:Socket_Strip_Angled_2x05 -> Pin_Headers:Pin_Header_Angled_2x05
Changed lines of the file:
@@
 F 0 "P2" H 9300 5500 50  0000 C CNN
 F 1 "Indicator Panel" H 9300 4900 50  0000 C CNN
-F 2 "Socket_Strips:Socket_Strip_Angled_2x05" H 9300 4000 50  0001 C CNN
+F 2 "Pin_Headers:Pin_Header_Angled_2x05" H 9300 4000 50  0001 C CNN
 F 3 "" H 9300 4000 50  0000 C CNN
 	1    9300 5200
@@
 $EndComp
 $Comp
-L GND #PWR0181
+L GND #PWR0138
 U 1 1 58C7C181
 P 8000 2300
-F 0 "#PWR0181" H 8000 2050 50  0001 C CNN
+F 0 "#PWR0138" H 8000 2050 50  0001 C CNN
 F 1 "GND" H 8000 2150 50  0001 C CNN
 F 2 "" H 8000 2300 50  0000 C CNN
@@
 	8000 2300 8000 2250
 $Comp
-L GND #PWR0182
+L GND #PWR0139
 U 1 1 58C7C5A9
 P 8200 2000
-F 0 "#PWR0182" H 8200 1750 50  0001 C CNN
+F 0 "#PWR0139" H 8200 1750 50  0001 C CNN
 F 1 "GND" H 8200 1850 50  0001 C CNN
 F 2 "" H 8200 2000 50  0000 C CNN
@@
 	8200 1700 8200 2000
 $Comp
-L +3V3 #PWR0183
+L +3V3 #PWR0140
 U 1 1 58C7C6E8
 P 8200 750
-F 0 "#PWR0183" H 8200 600 50  0001 C CNN
+F 0 "#PWR0140" H 8200 600 50  0001 C CNN
 F 1 "+3V3" H 8200 890 50  0000 C CNN
 F 2 "" H 8200 750 50  0000 C CNN
@@
 $EndComp
 $Comp
-L GND #PWR0184
+L GND #PWR0141
 U 1 1 58C7CFA0
 P 8000 4050
-F 0 "#PWR0184" H 8000 3800 50  0001 C CNN
+F 0 "#PWR0141" H 8000 3800 50  0001 C CNN
 F 1 "GND" H 8000 3900 50  0001 C CNN
 F 2 "" H 8000 4050 50  0000 C CNN
@@
 	8000 4050 8000 4000
 $Comp
-L GND #PWR0185
+L GND #PWR0142
 U 1 1 58C7CFC2
 P 8200 3750
-F 0 "#PWR0185" H 8200 3500 50  0001 C CNN
+F 0 "#PWR0142" H 8200 3500 50  0001 C CNN
 F 1 "GND" H 8200 3600 50  0001 C CNN
 F 2 "" H 8200 3750 50  0000 C CNN
@@
 	8200 3450 8200 3750
 $Comp
-L +3V3 #PWR0186
+L +3V3 #PWR0143
 U 1 1 58C7CFCA
 P 8200 2500
-F 0 "#PWR0186" H 8200 2350 50  0001 C CNN
+F 0 "#PWR0143" H 8200 2350 50  0001 C CNN
 F 1 "+3V3" H 8200 2640 50  0000 C CNN
 F 2 "" H 8200 2500 50  0000 C CNN
@@
 Connection ~ 8000 2550
 $Comp
-L GND #PWR0187
+L GND #PWR0144
 U 1 1 58C7DAE3
 P 10000 2200
-F 0 "#PWR0187" H 10000 1950 50  0001 C CNN
+F 0 "#PWR0144" H 10000 1950 50  0001 C CNN
 F 1 "GND" H 10000 2050 50  0001 C CNN
 F 2 "" H 10000 2200 50  0000 C CNN
@@
 $EndComp
 $Comp
-L GND #PWR0188
+L GND #PWR0145
 U 1 1 58C7DB1B
 P 10000 3950
-F 0 "#PWR0188" H 10000 3700 50  0001 C CNN
+F 0 "#PWR0145" H 10000 3700 50  0001 C CNN
 F 1 "GND" H 10000 3800 50  0001 C CNN
 F 2 "" H 10000 3950 50  0000 C CNN
@@
 	10000 2200 10000 2100
 $Comp
-L GND #PWR0189
+L GND #PWR0146
 U 1 1 58C7DE50
 P 5950 6450
-F 0 "#PWR0189" H 5950 6200 50  0001 C CNN
+F 0 "#PWR0146" H 5950 6200 50  0001 C CNN
 F 1 "GND" H 5950 6300 50  0001 C CNN
 F 2 "" H 5950 6450 50  0000 C CNN
@@
 	5500 5800 5550 5800
 $Comp
-L +5V_USB #PWR0190
+L +5V_USB #PWR0147
 U 1 1 58C7E0AF
 P 5500 5700
-F 0 "#PWR0190" H 5500 5550 50  0001 C CNN
+F 0 "#PWR0147" H 5500 5550 50  0001 C CNN
 F 1 "+5V_USB" H 5500 5840 50  0000 C CNN
 F 2 "" H 5500 5700 50  0000 C CNN
@@
 USB_D+
 $Comp
-L MAX3033E U601
-U 1 1 58C6D087
-P 7250 4650
-F 0 "U601" H 7800 4900 60  0000 C CNN
-F 1 "MAX3033E" H 7350 4900 60  0000 C CNN
-F 2 "Housings_SSOP:TSSOP-16_4.4x5mm_Pitch0.65mm" H 7250 4650 60  0001 C CNN
-F 3 "" H 7250 4650 60  0000 C CNN
-	1    7250 4650
-	1    0    0    -1
-$EndComp
-$Comp
-L +3V3 #PWR0191
+L +3V3 #PWR0148
 U 1 1 58C6D13C
 P 6950 4500
-F 0 "#PWR0191" H 6950 4350 50  0001 C CNN
+F 0 "#PWR0148" H 6950 4350 50  0001 C CNN
 F 1 "+3V3" H 6950 4640 50  0000 C CNN
 F 2 "" H 6950 4500 50  0000 C CNN
@@
 Connection ~ 5100 6100
 $Comp
-L GND #PWR0192
+L GND #PWR0149
 U 1 1 58C6CBD5
 P 5300 6450
-F 0 "#PWR0192" H 5300 6200 50  0001 C CNN
+F 0 "#PWR0149" H 5300 6200 50  0001 C CNN
 F 1 "GND" H 5300 6300 50  0001 C CNN
 F 2 "" H 5300 6450 50  0000 C CNN
@@
 $EndComp
 $Comp
-L GND #PWR0193
+L GND #PWR0150
 U 1 1 58C6CC16
 P 5100 6450
-F 0 "#PWR0193" H 5100 6200 50  0001 C CNN
+F 0 "#PWR0150" H 5100 6200 50  0001 C CNN
 F 1 "GND" H 5100 6300 50  0001 C CNN
 F 2 "" H 5100 6450 50  0000 C CNN
@@
 DIP_7
 $Comp
-L GND #PWR0194
+L GND #PWR0151
 U 1 1 58C72C63
 P 5950 3950
-F 0 "#PWR0194" H 5950 3700 50  0001 C CNN
+F 0 "#PWR0151" H 5950 3700 50  0001 C CNN
 F 1 "GND" H 5950 3800 50  0001 C CNN
 F 2 "" H 5950 3950 50  0000 C CNN
@@
 $EndComp
 $Comp
-L +3V3 #PWR0195
+L +3V3 #PWR0152
 U 1 1 58C74D20
 P 6100 800
-F 0 "#PWR0195" H 6100 650 50  0001 C CNN
+F 0 "#PWR0152" H 6100 650 50  0001 C CNN
 F 1 "+3V3" H 6100 940 50  0000 C CNN
 F 2 "" H 6100 800 50  0000 C CNN
@@
 	-1   0    0    -1
 $EndComp
+$Comp
+L MAX3033E U601
+U 1 1 5A4BF34B
+P 7250 4650
+F 0 "U601" H 7800 4900 60  0000 C CNN
+F 1 "MAX3033E" H 7350 4900 60  0000 C CNN
+F 2 "Housings_SSOP:TSSOP-16_4.4x5mm_Pitch0.65mm" H 7250 4650 60  0001 C CNN
+F 3 "" H 7250 4650 60  0000 C CNN
+	1    7250 4650
+	1    0    0    -1
+$EndComp
 $EndSCHEMATC

Commit message: Updated to KiCad v5
Parts:
- removed CON1: SD 0, myMods.pretty:microSD-3M-2900-series, symbol Micro_SD_Card
- removed CON2: SD 1, myMods.pretty:microSD-3M-2900-series, symbol Micro_SD_Card
- added CON1: SD 0, symbol qsic-rescue:Micro_SD_Card_Det
- added CON2: SD 1, symbol qsic-rescue:Micro_SD_Card_Det
- added U602: USB3340, Housings_DFN_QFN:QFN-32-1EP_5x5mm_Pitch0.5mm, symbol myLib:USB3340
- D601, D602, D603, D604, D605, D606, D607, D608: symbol LED_Small -> qsic-rescue:LED_Small
- J601: footprint (none) -> Connect:USB_A; symbol USB_A -> qsic-rescue:USB_A
- P2: symbol CONN_02X05 -> conn:CONN_02X05
- R601, R602, R603, R604, R605, R606, R607, R608, R609, R610, R611, R612, R613, R614, R615, R616, R617, R618, R619, R620: symbol R -> device:R
- S601: symbol DIP-Switch-8 -> myLib:DIP-Switch-8
- U401: symbol XC7A75T-CSG324 -> myLib:XC7A75T-CSG324
- U601: symbol MAX3033E -> myLib:MAX3033E
Connections:
- wire segments 81 -> 120
- no-connect marks 2 -> 0

Commit message: Updated to KiCad v5
Parts:
- P2: symbol conn:CONN_02X05 -> qsic-rescue:CONN_02X05-conn
- R601, R602, R603, R604, R605, R606, R607, R608, R609, R610, R611, R612, R613, R614, R615, R616, R617, R618, R619, R620: symbol device:R -> qsic-rescue:R-device
- U401: symbol myLib:XC7A75T-CSG324 -> qsic-rescue:XC7A75T-CSG324-myLib
- U602: symbol myLib:USB3340 -> qsic-rescue:USB3340-myLib
Changed lines of the file:
@@
 EESchema Schematic File Version 4
 LIBS:qsic-cache
-EELAYER 26 0
+EELAYER 30 0
 EELAYER END
 $Descr A 11000 8500
 encoding utf-8
-Sheet 6 6
+Sheet 7 7
 Title "I/O Ports"
 Date "2017-10-31"
@@
 $EndDescr
 $Comp
-L myLib:XC7A75T-CSG324 U401
+L qsic-rescue:XC7A75T-CSG324-myLib U401
 U 7 1 58C5DB74
 P 900 900
@@
 $EndComp
 $Comp
-L conn:CONN_02X05 P2
+L qsic-rescue:CONN_02X05-conn P2
 U 1 1 58C5E53F
 P 9300 5200
+AR Path="/58C5E53F" Ref="P2"  Part="1"
+AR Path="/58C5D743/58C5E53F" Ref="P2"  Part="1"
 F 0 "P2" H 9300 5500 50  0000 C CNN
 F 1 "Indicator Panel" H 9300 4900 50  0000 C CNN
@@
 $EndComp
 $Comp
-L device:R R613
+L qsic-rescue:R-device R613
 U 1 1 58C7BE06
 P 7600 1000
@@
 $EndComp
 $Comp
-L device:R R611
+L qsic-rescue:R-device R611
 U 1 1 58C76012
 P 7400 1000
@@
 $EndComp
 $Comp
-L device:R R615
+L qsic-rescue:R-device R615
 U 1 1 58C7BEA8
 P 7800 1000
@@
 $EndComp
 $Comp
-L device:R R617
+L qsic-rescue:R-device R617
 U 1 1 58C7BED4
 P 8000 1000
@@
 $EndComp
 $Comp
-L device:R R618
+L qsic-rescue:R-device R618
 U 1 1 58C7BF74
 P 8000 2100
@@
 Connection ~ 8000 800
 $Comp
-L device:R R614
+L qsic-rescue:R-device R614
 U 1 1 58C7CF7D
 P 7600 2750
@@
 $EndComp
 $Comp
-L device:R R612
+L qsic-rescue:R-device R612
 U 1 1 58C7CF84
 P 7400 2750
@@
 $EndComp
 $Comp
-L device:R R616
+L qsic-rescue:R-device R616
 U 1 1 58C7CF8B
 P 7800 2750
@@
 $EndComp
 $Comp
-L device:R R619
+L qsic-rescue:R-device R619
 U 1 1 58C7CF92
 P 8000 2750
@@
 $EndComp
 $Comp
-L device:R R620
+L qsic-rescue:R-device R620
 U 1 1 58C7CF99
 P 8000 3850
@@
 Connection ~ 6950 4550
 $Comp
-L device:R R602
+L qsic-rescue:R-device R602
 U 1 1 58C6C931
 P 5300 6300
@@
 $EndComp
 $Comp
-L device:R R601
+L qsic-rescue:R-device R601
 U 1 1 58C6C9B5
 P 5100 6300
@@
 $EndComp
 $Comp
-L device:R R603
+L qsic-rescue:R-device R603
 U 1 1 58C74888
 P 5800 900
@@
 $EndComp
 $Comp
-L device:R R604
+L qsic-rescue:R-device R604
 U 1 1 58C74923
 P 5800 1150
@@
 $EndComp
 $Comp
-L device:R R605
+L qsic-rescue:R-device R605
 U 1 1 58C74A8B
 P 5800 1400
@@
 $EndComp
 $Comp
-L device:R R606
+L qsic-rescue:R-device R606
 U 1 1 58C74A92
 P 5800 1650
@@
 $EndComp
 $Comp
-L device:R R607
+L qsic-rescue:R-device R607
 U 1 1 58C74B93
 P 5800 1900
@@
 $EndComp
 $Comp
-L device:R R608
+L qsic-rescue:R-device R608
 U 1 1 58C74B9A
 P 5800 2150
@@
 $EndComp
 $Comp
-L device:R R609
+L qsic-rescue:R-device R609
 U 1 1 58C74C56
 P 5800 2400
@@
 $EndComp
 $Comp
-L device:R R610
+L qsic-rescue:R-device R610
 U 1 1 58C74C5D
 P 5800 2650
@@
 $EndComp
 $Comp
-L myLib:USB3340 U602
+L qsic-rescue:USB3340-myLib U602
 U 1 1 5AC7CFB5
 P 3350 6800

Commit message: These are all old changes in directories that are now historical.
Parts:
- R601, R602, R603, R604, R605, R606, R607, R608, R609, R610, R611, R612, R613, R614, R615, R616, R617, R618, R619, R620: footprint Resistors_SMD:R_0603 -> Resistor_SMD:R_0603_1608Metric
Changed lines of the file:
@@
 EESchema Schematic File Version 4
-LIBS:qsic-cache
 EELAYER 30 0
 EELAYER END
 $Descr A 11000 8500
 encoding utf-8
-Sheet 7 7
+Sheet 7 8
 Title "I/O Ports"
 Date "2017-10-31"
@@
 F 0 "R613" V 7680 1000 50  0000 C CNN
 F 1 "50k" V 7600 1000 50  0000 C CNN
-F 2 "Resistors_SMD:R_0603" V 7530 1000 50  0001 C CNN
+F 2 "Resistor_SMD:R_0603_1608Metric" V 7530 1000 50  0001 C CNN
 F 3 "" H 7600 1000 50  0000 C CNN
 	1    7600 1000
@@
 F 0 "R611" V 7480 1000 50  0000 C CNN
 F 1 "50k" V 7400 1000 50  0000 C CNN
-F 2 "Resistors_SMD:R_0603" V 7330 1000 50  0001 C CNN
+F 2 "Resistor_SMD:R_0603_1608Metric" V 7330 1000 50  0001 C CNN
 F 3 "" H 7400 1000 50  0000 C CNN
 	1    7400 1000
@@
 F 0 "R615" V 7880 1000 50  0000 C CNN
 F 1 "50k" V 7800 1000 50  0000 C CNN
-F 2 "Resistors_SMD:R_0603" V 7730 1000 50  0001 C CNN
+F 2 "Resistor_SMD:R_0603_1608Metric" V 7730 1000 50  0001 C CNN
 F 3 "" H 7800 1000 50  0000 C CNN
 	1    7800 1000
@@
 F 0 "R617" V 8080 1000 50  0000 C CNN
 F 1 "50k" V 8000 1000 50  0000 C CNN
-F 2 "Resistors_SMD:R_0603" V 7930 1000 50  0001 C CNN
+F 2 "Resistor_SMD:R_0603_1608Metric" V 7930 1000 50  0001 C CNN
 F 3 "" H 8000 1000 50  0000 C CNN
 	1    8000 1000
@@
 F 0 "R618" V 8080 2100 50  0000 C CNN
 F 1 "270k" V 8000 2100 50  0000 C CNN
-F 2 "Resistors_SMD:R_0603" V 7930 2100 50  0001 C CNN
+F 2 "Resistor_SMD:R_0603_1608Metric" V 7930 2100 50  0001 C CNN
 F 3 "" H 8000 2100 50  0000 C CNN
 	1    8000 2100
@@
 F 0 "R614" V 7680 2750 50  0000 C CNN
 F 1 "50k" V 7600 2750 50  0000 C CNN
-F 2 "Resistors_SMD:R_0603" V 7530 2750 50  0001 C CNN
+F 2 "Resistor_SMD:R_0603_1608Metric" V 7530 2750 50  0001 C CNN
 F 3 "" H 7600 2750 50  0000 C CNN
 	1    7600 2750
@@
 F 0 "R612" V 7480 2750 50  0000 C CNN
 F 1 "50k" V 7400 2750 50  0000 C CNN
-F 2 "Resistors_SMD:R_0603" V 7330 2750 50  0001 C CNN
+F 2 "Resistor_SMD:R_0603_1608Metric" V 7330 2750 50  0001 C CNN
 F 3 "" H 7400 2750 50  0000 C CNN
 	1    7400 2750
@@
 F 0 "R616" V 7880 2750 50  0000 C CNN
 F 1 "50k" V 7800 2750 50  0000 C CNN
-F 2 "Resistors_SMD:R_0603" V 7730 2750 50  0001 C CNN
+F 2 "Resistor_SMD:R_0603_1608Metric" V 7730 2750 50  0001 C CNN
 F 3 "" H 7800 2750 50  0000 C CNN
 	1    7800 2750
@@
 F 0 "R619" V 8080 2750 50  0000 C CNN
 F 1 "50k" V 8000 2750 50  0000 C CNN
-F 2 "Resistors_SMD:R_0603" V 7930 2750 50  0001 C CNN
+F 2 "Resistor_SMD:R_0603_1608Metric" V 7930 2750 50  0001 C CNN
 F 3 "" H 8000 2750 50  0000 C CNN
 	1    8000 2750
@@
 F 0 "R620" V 8080 3850 50  0000 C CNN
 F 1 "270k" V 8000 3850 50  0000 C CNN
-F 2 "Resistors_SMD:R_0603" V 7930 3850 50  0001 C CNN
+F 2 "Resistor_SMD:R_0603_1608Metric" V 7930 3850 50  0001 C CNN
 F 3 "" H 8000 3850 50  0000 C CNN
 	1    8000 3850
@@
 F 0 "R602" V 5380 6300 50  0000 C CNN
 F 1 "15k" V 5300 6300 50  0000 C CNN
-F 2 "Resistors_SMD:R_0603" V 5230 6300 50  0001 C CNN
+F 2 "Resistor_SMD:R_0603_1608Metric" V 5230 6300 50  0001 C CNN
 F 3 "" H 5300 6300 50  0000 C CNN
 	1    5300 6300
@@
 F 0 "R601" V 5180 6300 50  0000 C CNN
 F 1 "15k" V 5100 6300 50  0000 C CNN
-F 2 "Resistors_SMD:R_0603" V 5030 6300 50  0001 C CNN
+F 2 "Resistor_SMD:R_0603_1608Metric" V 5030 6300 50  0001 C CNN
 F 3 "" H 5100 6300 50  0000 C CNN
 	1    5100 6300
@@
 F 0 "R603" V 5880 900 50  0000 C CNN
 F 1 "R" V 5800 900 50  0000 C CNN
-F 2 "Resistors_SMD:R_0603" V 5730 900 50  0001 C CNN
+F 2 "Resistor_SMD:R_0603_1608Metric" V 5730 900 50  0001 C CNN
 F 3 "" H 5800 900 50  0000 C CNN
 	1    5800 900
@@
 F 0 "R604" V 5880 1150 50  0000 C CNN
 F 1 "R" V 5800 1150 50  0000 C CNN
-F 2 "Resistors_SMD:R_0603" V 5730 1150 50  0001 C CNN
+F 2 "Resistor_SMD:R_0603_1608Metric" V 5730 1150 50  0001 C CNN
 F 3 "" H 5800 1150 50  0000 C CNN
 	1    5800 1150
@@
 F 0 "R605" V 5880 1400 50  0000 C CNN
 F 1 "R" V 5800 1400 50  0000 C CNN
-F 2 "Resistors_SMD:R_0603" V 5730 1400 50  0001 C CNN
+F 2 "Resistor_SMD:R_0603_1608Metric" V 5730 1400 50  0001 C CNN
 F 3 "" H 5800 1400 50  0000 C CNN
 	1    5800 1400
@@
 F 0 "R606" V 5880 1650 50  0000 C CNN
 F 1 "R" V 5800 1650 50  0000 C CNN
-F 2 "Resistors_SMD:R_0603" V 5730 1650 50  0001 C CNN
+F 2 "Resistor_SMD:R_0603_1608Metric" V 5730 1650 50  0001 C CNN
 F 3 "" H 5800 1650 50  0000 C CNN
 	1    5800 1650
@@
 F 0 "R607" V 5880 1900 50  0000 C CNN
 F 1 "R" V 5800 1900 50  0000 C CNN
-F 2 "Resistors_SMD:R_0603" V 5730 1900 50  0001 C CNN
+F 2 "Resistor_SMD:R_0603_1608Metric" V 5730 1900 50  0001 C CNN
 F 3 "" H 5800 1900 50  0000 C CNN
 	1    5800 1900
@@
 F 0 "R608" V 5880 2150 50  0000 C CNN
 F 1 "R" V 5800 2150 50  0000 C CNN
-F 2 "Resistors_SMD:R_0603" V 5730 2150 50  0001 C CNN
+F 2 "Resistor_SMD:R_0603_1608Metric" V 5730 2150 50  0001 C CNN
 F 3 "" H 5800 2150 50  0000 C CNN
 	1    5800 2150
@@
 F 0 "R609" V 5880 2400 50  0000 C CNN
 F 1 "R" V 5800 2400 50  0000 C CNN
-F 2 "Resistors_SMD:R_0603" V 5730 2400 50  0001 C CNN
+F 2 "Resistor_SMD:R_0603_1608Metric" V 5730 2400 50  0001 C CNN
 F 3 "" H 5800 2400 50  0000 C CNN
 	1    5800 2400
@@
 F 0 "R610" V 5880 2650 50  0000 C CNN
 F 1 "R" V 5800 2650 50  0000 C CNN
-F 2 "Resistors_SMD:R_0603" V 5730 2650 50  0001 C CNN
+F 2 "Resistor_SMD:R_0603_1608Metric" V 5730 2650 50  0001 C CNN
 F 3 "" H 5800 2650 50  0000 C CNN
 	1    5800 2650
