File: board-smt/memory.sch (KiCad schematic (older format))
At the start: 9 parts, among them U401 XC7A75T-CSG324, U501 IS43TR16128B

Commit message: Updated to KiCad v5
Parts:
- C501, C502: symbol C_Small -> device:C_Small
- R501, R502, R503, R504, R505: symbol R -> device:R
- U401: symbol XC7A75T-CSG324 -> myLib:XC7A75T-CSG324
- U501: symbol IS43TR16128B -> myLib:IS43TR16128B
Connections:
- wire segments 162 -> 205
Changed lines of the file:
@@
-EESchema Schematic File Version 2
-LIBS:qsic-rescue
-LIBS:power
-LIBS:device
-LIBS:transistors
-LIBS:conn
-LIBS:linear
-LIBS:regul
-LIBS:74xx
-LIBS:cmos4000
-LIBS:adc-dac
-LIBS:memory
-LIBS:xilinx
-LIBS:microcontrollers
-LIBS:dsp
-LIBS:microchip
-LIBS:analog_switches
-LIBS:motorola
-LIBS:texas
-LIBS:intel
-LIBS:audio
-LIBS:interface
-LIBS:digital-audio
-LIBS:philips
-LIBS:display
-LIBS:cypress
-LIBS:siliconi
-LIBS:opto
-LIBS:atmel
-LIBS:contrib
-LIBS:valves
-LIBS:myLib
+EESchema Schematic File Version 4
 LIBS:qsic-cache
-EELAYER 25 0
+EELAYER 26 0
 EELAYER END
 $Descr A 11000 8500
@@
 $EndDescr
 $Comp
-L XC7A75T-CSG324 U?
+L myLib:XC7A75T-CSG324 U?
 U 8 1 58C4BEB9
 P 800 800
@@
 $EndComp
 $Comp
-L IS43TR16128B U501
+L myLib:IS43TR16128B U501
 U 1 1 58C4BF43
 P 9800 2250
@@
 $EndComp
 $Comp
-L IS43TR16128B U501
+L myLib:IS43TR16128B U501
 U 2 1 58C4BFDC
 P 5550 1150
@@
 DQSU#
 $Comp
-L C_Small C501
+L device:C_Small C501
 U 1 1 58C4D47E
 P 3600 6100
@@
 $EndComp
 $Comp
-L C_Small C502
+L device:C_Small C502
 U 1 1 58C4D4C3
 P 3600 6550
@@
 $EndComp
 $Comp
-L R R503
+L device:R R503
 U 1 1 58C4D4F2
 P 3950 6100
@@
 $EndComp
 $Comp
-L R R504
+L device:R R504
 U 1 1 58C4D525
 P 3950 6550
@@
 $EndComp
 $Comp
-L +1V5 #PWR083
+L power:+1V5 #PWR083
 U 1 1 58C4D5AF
 P 3750 5850
@@
 $EndComp
 $Comp
-L R R502
+L device:R R502
 U 1 1 58C4DBA8
 P 3800 3500
@@
 $EndComp
 $Comp
-L R R505
+L device:R R505
 U 1 1 58C4DC41
 P 4100 3150
@@
 $EndComp
 $Comp
-L GND #PWR084
+L power:GND #PWR084
 U 1 1 58C4DCEE
 P 3900 3200
@@
 $EndComp
 $Comp
-L R R501
+L device:R R501
 U 1 1 58C4DD47
 P 3800 4000
@@
 $EndComp
 $Comp
-L GND #PWR085
+L power:GND #PWR085
 U 1 1 58C4DDD7
 P 3600 4050
@@
 	6550 3250 6650 3350
 $Comp
-L +1V5 #PWR086
+L power:+1V5 #PWR086
 U 1 1 58C4F4C4
 P 9100 2200
@@
 	-1   0    0    -1
 $EndComp
-Wire Bus Line
-	3000 650  3000 5850
-Wire Bus Line
-	3000 650  6650 650
-Wire Bus Line
-	6650 650  6650 3400
-Wire Bus Line
-	4350 750  4350 4800
 Wire Wire Line
 	2300 800  2900 800
@@
 	3950 6750 3950 6700
 Wire Wire Line
-	3600 6200 3600 6450
-Wire Wire Line
-	3950 6250 3950 6400
+	3600 6200 3600 6350
+Wire Wire Line
+	3950 6250 3950 6350
 Wire Wire Line
 	3600 6000 3600 5900
 Wire Wire Line
-	3600 5900 3950 5900
+	3600 5900 3750 5900
 Wire Wire Line
 	3950 5900 3950 5950
@@
 Connection ~ 3750 5900
 Wire Wire Line
-	2750 6350 3950 6350
+	2750 6350 3600 6350
 Connection ~ 3600 6350
 Connection ~ 3950 6350
 Wire Wire Line
-	2750 2000 2750 6350
+	2750 2000 2750 4600
 Wire Wire Line
 	2750 4600 2300 4600
@@
 	9100 3850 9200 3850
 Wire Wire Line
-	9100 2200 9100 3950
+	9100 2200 9100 2250
 Wire Wire Line
 	9100 3950 9200 3950
@@
 Connection ~ 9100 3850
 $Comp
-L GND #PWR087
+L power:GND #PWR087
 U 1 1 58C4FBDC
 P 9100 6200
@@
 	9100 6150 9200 6150
 Wire Wire Line
-	9100 4150 9100 6200
+	9100 4150 9100 4250
 Connection ~ 9100 4250
 Connection ~ 9100 4350
@@
 Connection ~ 9100 6150
 Wire Wire Line
-	8750 6350 9200 6350
+	8750 6350 9000 6350
 Wire Wire Line
 	9200 6450 9000 6450
@@
 VREF15
 $Comp
-L GND #PWR088
+L power:GND #PWR088
 U 1 1 58C75567
 P 3950 6750
@@
 $EndComp
 $Comp
-L GND #PWR089
+L power:GND #PWR089
 U 1 1 58C75590
 P 3600 6750
@@
 	-1   0    0    -1
 $EndComp
+Wire Wire Line
+	3750 5900 3950 5900
+Wire Wire Line
+	3600 6350 3600 6450
+Wire Wire Line
+	3600 6350 3950 6350
+Wire Wire Line
+	3950 6350 3950 6400
+Wire Wire Line
+	2750 4600 2750 6350
+Wire Wire Line
+	9100 2250 9100 2350
+Wire Wire Line
+	9100 2350 9100 2450
+Wire Wire Line
+	9100 2450 9100 2550
+Wire Wire Line
+	9100 2550 9100 2650
+Wire Wire Line
+	9100 2650 9100 2750
+Wire Wire Line
+	9100 2750 9100 2850
+Wire Wire Line
+	9100 2850 9100 2950
+Wire Wire Line
+	9100 2950 9100 3050
+Wire Wire Line
+	9100 3050 9100 3150
+Wire Wire Line
+	9100 3150 9100 3250
+Wire Wire Line
+	9100 3250 9100 3350
+Wire Wire Line
+	9100 3350 9100 3450
+Wire Wire Line
+	9100 3450 9100 3550
+Wire Wire Line
+	9100 3550 9100 3650
+Wire Wire Line
+	9100 3650 9100 3750
+Wire Wire Line
+	9100 3750 9100 3850
+Wire Wire Line
+	9100 3850 9100 3950
+Wire Wire Line
+	9100 4250 9100 4350
+Wire Wire Line
+	9100 4350 9100 4450
+Wire Wire Line
+	9100 4450 9100 4550
+Wire Wire Line
+	9100 4550 9100 4650
+Wire Wire Line
+	9100 4650 9100 4750
+Wire Wire Line
+	9100 4750 9100 4850
+Wire Wire Line
+	9100 4850 9100 4950
+Wire Wire Line
+	9100 4950 9100 5050
+Wire Wire Line
+	9100 5050 9100 5150
+Wire Wire Line
+	9100 5150 9100 5250
+Wire Wire Line
+	9100 5250 9100 5350
+Wire Wire Line
+	9100 5350 9100 5450
+Wire Wire Line
+	9100 5450 9100 5550
+Wire Wire Line
+	9100 5550 9100 5650
+Wire Wire Line
+	9100 5650 9100 5750
+Wire Wire Line
+	9100 5750 9100 5850
+Wire Wire Line
+	9100 5850 9100 5950
+Wire Wire Line
+	9100 5950 9100 6050
+Wire Wire Line
+	9100 6050 9100 6150
+Wire Wire Line
+	9100 6150 9100 6200
+Wire Wire Line
+	9000 6350 9200 6350
+Wire Bus Line
+	3000 650  6650 650
+Wire Bus Line
+	6650 650  6650 3400
+Wire Bus Line
+	4350 750  4350 4800
+Wire Bus Line
+	3000 650  3000 5850
 $EndSCHEMATC

Commit message: Updated to KiCad v5
Parts:
- C501, C502: symbol device:C_Small -> qsic-rescue:C_Small-device
- R501, R502, R503, R504, R505: symbol device:R -> qsic-rescue:R-device
- U401: symbol myLib:XC7A75T-CSG324 -> qsic-rescue:XC7A75T-CSG324-myLib
Changed lines of the file:
@@
 EESchema Schematic File Version 4
 LIBS:qsic-cache
-EELAYER 26 0
+EELAYER 30 0
 EELAYER END
 $Descr A 11000 8500
 encoding utf-8
-Sheet 4 6
+Sheet 4 7
 Title "Memory"
 Date "2017-10-31"
@@
 $EndDescr
 $Comp
-L myLib:XC7A75T-CSG324 U?
+L qsic-rescue:XC7A75T-CSG324-myLib U?
 U 8 1 58C4BEB9
 P 800 800
@@
 DQSU#
 $Comp
-L device:C_Small C501
+L qsic-rescue:C_Small-device C501
 U 1 1 58C4D47E
 P 3600 6100
@@
 $EndComp
 $Comp
-L device:C_Small C502
+L qsic-rescue:C_Small-device C502
 U 1 1 58C4D4C3
 P 3600 6550
@@
 $EndComp
 $Comp
-L device:R R503
+L qsic-rescue:R-device R503
 U 1 1 58C4D4F2
 P 3950 6100
@@
 $EndComp
 $Comp
-L device:R R504
+L qsic-rescue:R-device R504
 U 1 1 58C4D525
 P 3950 6550
@@
 $EndComp
 $Comp
-L device:R R502
+L qsic-rescue:R-device R502
 U 1 1 58C4DBA8
 P 3800 3500
@@
 $EndComp
 $Comp
-L device:R R505
+L qsic-rescue:R-device R505
 U 1 1 58C4DC41
 P 4100 3150
@@
 $EndComp
 $Comp
-L device:R R501
+L qsic-rescue:R-device R501
 U 1 1 58C4DD47
 P 3800 4000

Commit message: These are all old changes in directories that are now historical.
Parts:
- R501, R502, R503, R504, R505: footprint Resistors_SMD:R_0603 -> Resistor_SMD:R_0603_1608Metric
Changed lines of the file:
@@
 EESchema Schematic File Version 4
-LIBS:qsic-cache
 EELAYER 30 0
 EELAYER END
 $Descr A 11000 8500
 encoding utf-8
-Sheet 4 7
+Sheet 5 8
 Title "Memory"
 Date "2017-10-31"
@@
 F 0 "R503" V 4030 6100 50  0000 C CNN
 F 1 "47" V 3950 6100 50  0000 C CNN
-F 2 "Resistors_SMD:R_0603" V 3880 6100 50  0001 C CNN
+F 2 "Resistor_SMD:R_0603_1608Metric" V 3880 6100 50  0001 C CNN
 F 3 "" H 3950 6100 50  0000 C CNN
 	1    3950 6100
@@
 F 0 "R504" V 4030 6550 50  0000 C CNN
 F 1 "47" V 3950 6550 50  0000 C CNN
-F 2 "Resistors_SMD:R_0603" V 3880 6550 50  0001 C CNN
+F 2 "Resistor_SMD:R_0603_1608Metric" V 3880 6550 50  0001 C CNN
 F 3 "" H 3950 6550 50  0000 C CNN
 	1    3950 6550
@@
 F 0 "R502" V 3880 3500 50  0000 C CNN
 F 1 "89" V 3800 3500 50  0000 C CNN
-F 2 "Resistors_SMD:R_0603" V 3730 3500 50  0001 C CNN
+F 2 "Resistor_SMD:R_0603_1608Metric" V 3730 3500 50  0001 C CNN
 F 3 "" H 3800 3500 50  0000 C CNN
 	1    3800 3500
@@
 F 0 "R505" V 4180 3150 50  0000 C CNN
 F 1 "240" V 4100 3150 50  0000 C CNN
-F 2 "Resistors_SMD:R_0603" V 4030 3150 50  0001 C CNN
+F 2 "Resistor_SMD:R_0603_1608Metric" V 4030 3150 50  0001 C CNN
 F 3 "" H 4100 3150 50  0000 C CNN
 	1    4100 3150
@@
 F 0 "R501" V 3880 4000 50  0000 C CNN
 F 1 "47k" V 3800 4000 50  0000 C CNN
-F 2 "Resistors_SMD:R_0603" V 3730 4000 50  0001 C CNN
+F 2 "Resistor_SMD:R_0603_1608Metric" V 3730 4000 50  0001 C CNN
 F 3 "" H 3800 4000 50  0000 C CNN
 	1    3800 4000
