File: board-smt/power.sch (KiCad schematic (older format))
At the start: 3 parts, among them U401 XC7A75T-CSG324

Commit message: Added some voltage regulators.
Parts:
- added C301, C302, C309, C310: 10uF, Capacitors_SMD:C_0603, symbol C_Small
- added C303, C304: 2.2nF, Capacitors_SMD:C_0603, symbol C_Small
- added C305, C306, C311, C312: 100nF, Capacitors_SMD:C_0603, symbol C_Small
- added C307, C308, C313, C314: 22uF, Capacitors_SMD:C_0805, symbol C_Small
- added L301, L302: 4.7uH, Resistors_SMD:R_0805, symbol L_Small
- added L303: 1.5uH, Resistors_SMD:R_0805, symbol L_Small
- added L304: 2.2uH, Resistors_SMD:R_0805, symbol L_Small
- added R362, R363: 7.5k, Resistors_SMD:R_0603, symbol R
- added R364: 31.1k, Resistors_SMD:R_0603, symbol R
- added R365, R366: 10k, Resistors_SMD:R_0603, symbol R
- added R367: 11.5k, Resistors_SMD:R_0603, symbol R
- added R368: 100k, Resistors_SMD:R_0603, symbol R
- added R369: 50k, Resistors_SMD:R_0603, symbol R
- added R370: 18.2k, Resistors_SMD:R_0603, symbol R
- added R371: 4.7k, Resistors_SMD:R_0603, symbol R
- added U306, U307: AOZ3010PI, Housings_SOIC:SOIC-8-1EP_3.9x4.9mm_Pitch1.27mm, symbol AOZ3010PI
- added U308: RT8288A, Housings_SOIC:SOIC-8-1EP_3.9x4.9mm_Pitch1.27mm, symbol RT8288A
- added U309: SC189, TO_SOT_Packages_SMD:SOT-23-5, symbol SC189
Connections:
- net labels added: +5V
- wire segments 108 -> 180
Other:
- note added: "1.0V/4A"
- note added: "1.5V/2A"
- note added: "1.8V/1.5A"
- note added: "3.3V/2A"

Commit message: Moved comparator power connections to separate symbols.
Parts:
- added C315, C316, C317, C318, C319, C320, C321, C322, C323, C324, C325, C326: 100nF, Capacitors_SMD:C_0603, symbol C_Small
- added U201, U202, U203, U204, U205, U206, U301, U302, U303, U304, U305: CMP401, Housings_SOIC:SOIC-16_3.9x9.9mm_Pitch1.27mm, symbol CMP401
Connections:
- wire segments 180 -> 411

Commit message: Little fixups
Connections:
- wire segments 411 -> 233

Commit message: Updated to KiCad v5
Parts:
- C301, C302, C303, C304, C305, C306, C307, C308, C309, C310, C311, C312, C313, C314, C315, C316, C317, C318, C319, C320, C321, C322, C323, C324, C325, C326: symbol C_Small -> device:C_Small
- D301: value LED_Small_ALT -> Configure; symbol LED_Small_ALT -> qsic-rescue:LED_Small_ALT
- L301, L302, L303, L304: symbol L_Small -> device:L_Small
- R361, R362, R363, R364, R365, R366, R367, R368, R369, R370, R371: symbol R -> device:R
- U201, U202, U203, U204, U205, U206, U301, U302, U303, U304, U305: symbol CMP401 -> myLib:CMP401
- U306, U307: symbol AOZ3010PI -> myLib:AOZ3010PI
- U308: symbol RT8288A -> myLib:RT8288A
- U309: symbol SC189 -> myLib:SC189
- U401: symbol XC7A75T-CSG324 -> myLib:XC7A75T-CSG324
Connections:
- wire segments 233 -> 412

Commit message: Updated to KiCad v5
Parts:
- C301, C302, C303, C304, C305, C306, C307, C308, C309, C310, C311, C312, C313, C314, C315, C316, C317, C318, C319, C320, C321, C322, C323, C324, C325, C326: symbol device:C_Small -> qsic-rescue:C_Small-device
- L301, L302, L303, L304: symbol device:L_Small -> qsic-rescue:L_Small-device
- R361, R362, R363, R364, R365, R366, R367, R368, R369, R370, R371: symbol device:R -> qsic-rescue:R-device
- U401: symbol myLib:XC7A75T-CSG324 -> qsic-rescue:XC7A75T-CSG324-myLib
Changed lines of the file:
@@
 EESchema Schematic File Version 4
 LIBS:qsic-cache
-EELAYER 26 0
+EELAYER 30 0
 EELAYER END
 $Descr A 11000 8500
 encoding utf-8
-Sheet 3 6
+Sheet 3 7
 Title "Power"
 Date "2017-10-31"
@@
 Connection ~ 1750 3100
 $Comp
-L myLib:XC7A75T-CSG324 U401
+L qsic-rescue:XC7A75T-CSG324-myLib U401
 U 1 1 58C48354
 P 850 3000
@@
 $EndComp
 $Comp
-L myLib:XC7A75T-CSG324 U401
+L qsic-rescue:XC7A75T-CSG324-myLib U401
 U 2 1 58C483A8
 P 3550 5600
@@
 $EndComp
 $Comp
-L myLib:XC7A75T-CSG324 U401
+L qsic-rescue:XC7A75T-CSG324-myLib U401
 U 3 1 58C48929
 P 2100 4600
@@
 $EndComp
 $Comp
-L myLib:XC7A75T-CSG324 U401
+L qsic-rescue:XC7A75T-CSG324-myLib U401
 U 6 1 58C48AE5
 P 8900 5650
@@
 $EndComp
 $Comp
-L myLib:XC7A75T-CSG324 U401
+L qsic-rescue:XC7A75T-CSG324-myLib U401
 U 9 1 58C73D0A
 P 10000 1100
@@
 $EndComp
 $Comp
-L device:R R361
+L qsic-rescue:R-device R361
 U 1 1 58C74362
 P 8700 2050
@@
 $EndComp
 $Comp
-L device:C_Small C305
+L qsic-rescue:C_Small-device C305
 U 1 1 58F8DB21
 P 3250 800
@@
 $EndComp
 $Comp
-L device:C_Small C301
+L qsic-rescue:C_Small-device C301
 U 1 1 58F8DBBA
 P 2200 1350
@@
 $EndComp
 $Comp
-L device:C_Small C303
+L qsic-rescue:C_Small-device C303
 U 1 1 58F8DC45
 P 2350 1850
@@
 $EndComp
 $Comp
-L device:R R362
+L qsic-rescue:R-device R362
 U 1 1 58F8DC8E
 P 2350 1550
@@
 $EndComp
 $Comp
-L device:L_Small L301
+L qsic-rescue:L_Small-device L301
 U 1 1 58F8DDF4
 P 3750 1200
@@
 $EndComp
 $Comp
-L device:R R364
+L qsic-rescue:R-device R364
 U 1 1 58F8DE54
 P 3900 1350
@@
 $EndComp
 $Comp
-L device:R R365
+L qsic-rescue:R-device R365
 U 1 1 58F8DEA3
 P 3900 1700
@@
 $EndComp
 $Comp
-L device:C_Small C307
+L qsic-rescue:C_Small-device C307
 U 1 1 58F8DEFF
 P 4150 1350
@@
 $EndComp
 $Comp
-L device:C_Small C306
+L qsic-rescue:C_Small-device C306
 U 1 1 58F91031
 P 3250 2400
@@
 $EndComp
 $Comp
-L device:C_Small C302
+L qsic-rescue:C_Small-device C302
 U 1 1 58F9103E
 P 2200 2950
@@
 $EndComp
 $Comp
-L device:C_Small C304
+L qsic-rescue:C_Small-device C304
 U 1 1 58F91045
 P 2350 3450
@@
 $EndComp
 $Comp
-L device:R R363
+L qsic-rescue:R-device R363
 U 1 1 58F9104C
 P 2350 3150
@@
 $EndComp
 $Comp
-L device:L_Small L302
+L qsic-rescue:L_Small-device L302
 U 1 1 58F91053
 P 3750 2800
@@
 $EndComp
 $Comp
-L device:R R366
+L qsic-rescue:R-device R366
 U 1 1 58F9105A
 P 3900 2950
@@
 $EndComp
 $Comp
-L device:R R367
+L qsic-rescue:R-device R367
 U 1 1 58F91061
 P 3900 3300
@@
 $EndComp
 $Comp
-L device:C_Small C308
+L qsic-rescue:C_Small-device C308
 U 1 1 58F91068
 P 4150 2950
@@
 1.0V/4A
 $Comp
-L device:C_Small C309
+L qsic-rescue:C_Small-device C309
 U 1 1 58F92266
 P 5200 3050
@@
 $EndComp
 $Comp
-L device:C_Small C311
+L qsic-rescue:C_Small-device C311
 U 1 1 58F924B9
 P 6500 2700
@@
 $EndComp
 $Comp
-L device:R R369
+L qsic-rescue:R-device R369
 U 1 1 58F925C5
 P 6600 3200
@@
 $EndComp
 $Comp
-L device:R R371
+L qsic-rescue:R-device R371
 U 1 1 58F9266F
 P 7000 3200
@@
 $EndComp
 $Comp
-L device:R R370
+L qsic-rescue:R-device R370
 U 1 1 58F92727
 P 6800 3400
@@
 $EndComp
 $Comp
-L device:C_Small C312
+L qsic-rescue:C_Small-device C312
 U 1 1 58F92807
 P 6500 3500
@@
 $EndComp
 $Comp
-L device:C_Small C314
+L qsic-rescue:C_Small-device C314
 U 1 1 58F928CD
 P 7250 3350
@@
 $EndComp
 $Comp
-L device:R R368
+L qsic-rescue:R-device R368
 U 1 1 58F929A0
 P 5400 2850
@@
 $EndComp
 $Comp
-L device:L_Small L304
+L qsic-rescue:L_Small-device L304
 U 1 1 58F96B5E
 P 6850 3000
@@
 $EndComp
 $Comp
-L device:L_Small L303
+L qsic-rescue:L_Small-device L303
 U 1 1 58F97BE7
 P 6450 1350
@@
 $EndComp
 $Comp
-L device:C_Small C313
+L qsic-rescue:C_Small-device C313
 U 1 1 58F980E5
 P 6650 1600
@@
 $EndComp
 $Comp
-L device:C_Small C310
+L qsic-rescue:C_Small-device C310
 U 1 1 58F987CF
 P 5300 1600
@@
 Connection ~ 6650 1750
 $Comp
-L device:C_Small C317
+L qsic-rescue:C_Small-device C317
 U 1 1 5901272D
 P 7800 5950
@@
 $EndComp
 $Comp
-L device:C_Small C320
+L qsic-rescue:C_Small-device C320
 U 1 1 59012C9B
 P 8050 5950
@@
 Connection ~ 7800 5850
 $Comp
-L device:C_Small C323
+L qsic-rescue:C_Small-device C323
 U 1 1 59012FF2
 P 8300 5950
@@
 $EndComp
 $Comp
-L device:C_Small C326
+L qsic-rescue:C_Small-device C326
 U 1 1 59013086
 P 8550 5950
@@
 Connection ~ 8050 6050
 $Comp
-L device:C_Small C315
+L qsic-rescue:C_Small-device C315
 U 1 1 59013940
 P 7750 5350
@@
 $EndComp
 $Comp
-L device:C_Small C318
+L qsic-rescue:C_Small-device C318
 U 1 1 59013947
 P 8000 5350
@@
 Connection ~ 7750 5250
 $Comp
-L device:C_Small C321
+L qsic-rescue:C_Small-device C321
 U 1 1 59013950
 P 8250 5350
@@
 $EndComp
 $Comp
-L device:C_Small C324
+L qsic-rescue:C_Small-device C324
 U 1 1 59013957
 P 8500 5350
@@
 Connection ~ 8000 5450
 $Comp
-L device:C_Small C316
+L qsic-rescue:C_Small-device C316
 U 1 1 59013ABE
 P 7750 6400
@@
 $EndComp
 $Comp
-L device:C_Small C319
+L qsic-rescue:C_Small-device C319
 U 1 1 59013AC5
 P 8000 6400
@@
 Connection ~ 7750 6300
 $Comp
-L device:C_Small C322
+L qsic-rescue:C_Small-device C322
 U 1 1 59013ACE
 P 8250 6400
@@
 $EndComp
 $Comp
-L device:C_Small C325
+L qsic-rescue:C_Small-device C325
 U 1 1 59013AD5
 P 8500 6400

Commit message: These are all old changes in directories that are now historical.
Parts:
- R361, R362, R363, R364, R365, R366, R367, R368, R369, R370, R371: footprint Resistors_SMD:R_0603 -> Resistor_SMD:R_0603_1608Metric
Changed lines of the file:
@@
 EESchema Schematic File Version 4
-LIBS:qsic-cache
 EELAYER 30 0
 EELAYER END
 $Descr A 11000 8500
 encoding utf-8
-Sheet 3 7
+Sheet 4 8
 Title "Power"
 Date "2017-10-31"
@@
 F 0 "R361" V 8780 2050 50  0000 C CNN
 F 1 "240" V 8700 2050 50  0000 C CNN
-F 2 "Resistors_SMD:R_0603" V 8630 2050 50  0001 C CNN
+F 2 "Resistor_SMD:R_0603_1608Metric" V 8630 2050 50  0001 C CNN
 F 3 "" H 8700 2050 50  0000 C CNN
 	1    8700 2050
@@
 F 0 "R362" V 2430 1550 50  0000 C CNN
 F 1 "7.5k" V 2350 1550 50  0000 C CNN
-F 2 "Resistors_SMD:R_0603" V 2280 1550 50  0001 C CNN
+F 2 "Resistor_SMD:R_0603_1608Metric" V 2280 1550 50  0001 C CNN
 F 3 "" H 2350 1550 50  0000 C CNN
 	1    2350 1550
@@
 F 0 "R364" V 3980 1350 50  0000 C CNN
 F 1 "31.1k" V 3900 1350 50  0000 C CNN
-F 2 "Resistors_SMD:R_0603" V 3830 1350 50  0001 C CNN
+F 2 "Resistor_SMD:R_0603_1608Metric" V 3830 1350 50  0001 C CNN
 F 3 "" H 3900 1350 50  0000 C CNN
 	1    3900 1350
@@
 F 0 "R365" V 3980 1700 50  0000 C CNN
 F 1 "10k" V 3900 1700 50  0000 C CNN
-F 2 "Resistors_SMD:R_0603" V 3830 1700 50  0001 C CNN
+F 2 "Resistor_SMD:R_0603_1608Metric" V 3830 1700 50  0001 C CNN
 F 3 "" H 3900 1700 50  0000 C CNN
 	1    3900 1700
@@
 F 0 "R363" V 2430 3150 50  0000 C CNN
 F 1 "7.5k" V 2350 3150 50  0000 C CNN
-F 2 "Resistors_SMD:R_0603" V 2280 3150 50  0001 C CNN
+F 2 "Resistor_SMD:R_0603_1608Metric" V 2280 3150 50  0001 C CNN
 F 3 "" H 2350 3150 50  0000 C CNN
 	1    2350 3150
@@
 F 0 "R366" V 3980 2950 50  0000 C CNN
 F 1 "10k" V 3900 2950 50  0000 C CNN
-F 2 "Resistors_SMD:R_0603" V 3830 2950 50  0001 C CNN
+F 2 "Resistor_SMD:R_0603_1608Metric" V 3830 2950 50  0001 C CNN
 F 3 "" H 3900 2950 50  0000 C CNN
 	1    3900 2950
@@
 F 0 "R367" V 3980 3300 50  0000 C CNN
 F 1 "11.5k" V 3900 3300 50  0000 C CNN
-F 2 "Resistors_SMD:R_0603" V 3830 3300 50  0001 C CNN
+F 2 "Resistor_SMD:R_0603_1608Metric" V 3830 3300 50  0001 C CNN
 F 3 "" H 3900 3300 50  0000 C CNN
 	1    3900 3300
@@
 F 0 "R369" V 6680 3200 50  0000 C CNN
 F 1 "50k" V 6600 3200 50  0000 C CNN
-F 2 "Resistors_SMD:R_0603" V 6530 3200 50  0001 C CNN
+F 2 "Resistor_SMD:R_0603_1608Metric" V 6530 3200 50  0001 C CNN
 F 3 "" H 6600 3200 50  0000 C CNN
 	1    6600 3200
@@
 F 0 "R371" V 7080 3200 50  0000 C CNN
 F 1 "4.7k" V 7000 3200 50  0000 C CNN
-F 2 "Resistors_SMD:R_0603" V 6930 3200 50  0001 C CNN
+F 2 "Resistor_SMD:R_0603_1608Metric" V 6930 3200 50  0001 C CNN
 F 3 "" H 7000 3200 50  0000 C CNN
 	1    7000 3200
@@
 F 0 "R370" V 6880 3400 50  0000 C CNN
 F 1 "18.2k" V 6800 3400 50  0000 C CNN
-F 2 "Resistors_SMD:R_0603" V 6730 3400 50  0001 C CNN
+F 2 "Resistor_SMD:R_0603_1608Metric" V 6730 3400 50  0001 C CNN
 F 3 "" H 6800 3400 50  0000 C CNN
 	1    6800 3400
@@
 F 0 "R368" V 5480 2850 50  0000 C CNN
 F 1 "100k" V 5400 2850 50  0000 C CNN
-F 2 "Resistors_SMD:R_0603" V 5330 2850 50  0001 C CNN
+F 2 "Resistor_SMD:R_0603_1608Metric" V 5330 2850 50  0001 C CNN
 F 3 "" H 5400 2850 50  0000 C CNN
 	1    5400 2850
