File: board-smt/qsic.sch (KiCad schematic (older format))
At the start: 1 part

Commit message: Added board-prototype.
Connections:
- net labels removed: +12V, -12V
- wire segments 18 -> 12
- no-connect marks 0 -> 15
Changed lines of the file:
@@
 	0    1    1    0
 $EndComp
-$Comp
-L +12V #PWR03
-U 1 1 56137ADC
-P 15900 3600
-F 0 "#PWR03" H 15900 3450 50  0001 C CNN
-F 1 "+12V" H 15900 3740 50  0000 C CNN
-F 2 "" H 15900 3600 60  0000 C CNN
-F 3 "" H 15900 3600 60  0000 C CNN
-	1    15900 3600
-	0    1    1    0
-$EndComp
-$Comp
-L -12V #PWR102
-U 1 1 56137AF4
-P 15900 3800
-F 0 "#PWR102" H 15900 3900 50  0001 C CNN
-F 1 "-12V" H 15900 3950 50  0000 C CNN
-F 2 "" H 15900 3800 60  0000 C CNN
-F 3 "" H 15900 3800 60  0000 C CNN
-	1    15900 3800
-	0    1    1    0
-$EndComp
-Wire Wire Line
-	15800 3700 15900 3700
-Wire Wire Line
-	15900 3700 15900 3600
-Wire Wire Line
-	15900 3600 15800 3600
-Wire Wire Line
-	15800 3800 15900 3800
-Wire Wire Line
-	15800 3900 15900 3900
-Wire Wire Line
-	15900 3900 15900 3800
 Wire Wire Line
 	15800 4000 15900 4000
@@
 Connection ~ 15900 4100
 $Comp
-L PWR_FLAG #FLG04
-U 1 1 56137CC3
-P 14450 6350
-F 0 "#FLG04" H 14450 6445 50  0001 C CNN
-F 1 "PWR_FLAG" H 14450 6530 50  0000 C CNN
-F 2 "" H 14450 6350 60  0000 C CNN
-F 3 "" H 14450 6350 60  0000 C CNN
-	1    14450 6350
-	1    0    0    -1
-$EndComp
-$Comp
-L +12V #PWR05
-U 1 1 56137D2A
-P 14450 6350
-F 0 "#PWR05" H 14450 6200 50  0001 C CNN
-F 1 "+12V" H 14450 6490 50  0000 C CNN
-F 2 "" H 14450 6350 60  0000 C CNN
-F 3 "" H 14450 6350 60  0000 C CNN
-	1    14450 6350
-	-1   0    0    1
-$EndComp
-$Comp
-L PWR_FLAG #FLG06
-U 1 1 56137D69
-P 14900 6350
-F 0 "#FLG06" H 14900 6445 50  0001 C CNN
-F 1 "PWR_FLAG" H 14900 6530 50  0000 C CNN
-F 2 "" H 14900 6350 60  0000 C CNN
-F 3 "" H 14900 6350 60  0000 C CNN
-	1    14900 6350
-	1    0    0    -1
-$EndComp
-$Comp
-L PWR_FLAG #FLG07
+L PWR_FLAG #FLG03
 U 1 1 56137D79
 P 15350 6350
-F 0 "#FLG07" H 15350 6445 50  0001 C CNN
+F 0 "#FLG03" H 15350 6445 50  0001 C CNN
 F 1 "PWR_FLAG" H 15350 6530 50  0000 C CNN
 F 2 "" H 15350 6350 60  0000 C CNN
@@
 $EndComp
 $Comp
-L PWR_FLAG #FLG08
+L PWR_FLAG #FLG04
 U 1 1 56137D87
 P 15800 6350
-F 0 "#FLG08" H 15800 6445 50  0001 C CNN
+F 0 "#FLG04" H 15800 6445 50  0001 C CNN
 F 1 "PWR_FLAG" H 15800 6530 50  0000 C CNN
 F 2 "" H 15800 6350 60  0000 C CNN
@@
 $EndComp
 $Comp
-L -12V #PWR106
-U 1 1 56137D96
-P 14900 6350
-F 0 "#PWR106" H 14900 6450 50  0001 C CNN
-F 1 "-12V" H 14900 6500 50  0000 C CNN
-F 2 "" H 14900 6350 60  0000 C CNN
-F 3 "" H 14900 6350 60  0000 C CNN
-	1    14900 6350
-	-1   0    0    1
-$EndComp
-$Comp
-L +5V #PWR09
+L +5V #PWR05
 U 1 1 56137DA4
 P 15350 6350
-F 0 "#PWR09" H 15350 6200 50  0001 C CNN
+F 0 "#PWR05" H 15350 6200 50  0001 C CNN
 F 1 "+5V" H 15350 6490 50  0000 C CNN
 F 2 "" H 15350 6350 60  0000 C CNN
@@
 $EndComp
 $Comp
-L GND #PWR010
+L GND #PWR06
 U 1 1 56137DB2
 P 15800 6350
-F 0 "#PWR010" H 15800 6100 50  0001 C CNN
+F 0 "#PWR06" H 15800 6100 50  0001 C CNN
 F 1 "GND" H 15800 6200 50  0000 C CNN
 F 2 "" H 15800 6350 60  0000 C CNN
@@
 Text GLabel 14150 4050 0    60   Input ~ 0
 BDOUT
+NoConn ~ 15800 3600
+NoConn ~ 15800 3700
+NoConn ~ 15800 3800
+NoConn ~ 15800 3900
+NoConn ~ 15800 3250
+NoConn ~ 15800 3150
+NoConn ~ 15800 3050
+NoConn ~ 15800 2950
+NoConn ~ 15800 2850
+NoConn ~ 15800 2300
+NoConn ~ 15800 2200
+NoConn ~ 15800 2100
+NoConn ~ 15800 2000
+NoConn ~ 15800 1900
+NoConn ~ 15800 1800
 $EndSCHEMATC

Commit message: Added bus termination.
Parts:
- removed B101: QBus, myMods.pretty:Qbus-double, symbol QBus
Connections:
- net labels removed: BBS7, BDAL0, BDAL1, BDAL10, BDAL11, BDAL12, BDAL13, BDAL14, BDAL15, BDAL16, BDAL17, BDAL18, BDAL19, BDAL2, BDAL20, BDAL21, BDAL3, BDAL4, BDAL5, BDAL6, BDAL7, BDAL8, BDAL9, BDCOK, BDIN, BDMGI, BDMGO, BDMR, BDOUT, BEVNT, BHALT, BIAKI, BIAKO, BINIT, BIRQ4, BIRQ5, BIRQ6, BIRQ7, BPOK, BREF, BRPLY, BSACK, BSYNC, BWTBT
- wire segments 12 -> 0
- no-connect marks 15 -> 0
Changed lines of the file:
@@
 Comment4 ""
 $EndDescr
-$Comp
-L QBus B101
-U 1 1 560C3E74
-P 15600 3600
-F 0 "B101" H 15025 3400 60  0000 C CNN
-F 1 "QBus" H 15025 3175 60  0000 C CNN
-F 2 "myMods.pretty:Qbus-double" H 15600 3600 60  0001 C CNN
-F 3 "" H 15600 3600 60  0000 C CNN
-	1    15600 3600
-	1    0    0    -1
-$EndComp
-Text GLabel 14150 5050 0    60   Input ~ 0
-BSACK
-Text GLabel 14150 4850 0    60   Input ~ 0
-BDMGI
-Text GLabel 14150 4950 0    60   Input ~ 0
-BDMGO
 $Sheet
 S 11550 3900 900  2350
@@
 F1 "drivers.sch" 60
 $EndSheet
-Text GLabel 14150 1500 0    60   Input ~ 0
-BDAL0
-Text GLabel 14150 1600 0    60   Input ~ 0
-BDAL1
-Text GLabel 14150 1700 0    60   Input ~ 0
-BDAL2
-Text GLabel 14150 1800 0    60   Input ~ 0
-BDAL3
-Text GLabel 14150 1900 0    60   Input ~ 0
-BDAL4
-Text GLabel 14150 2000 0    60   Input ~ 0
-BDAL5
-Text GLabel 14150 2100 0    60   Input ~ 0
-BDAL6
-Text GLabel 14150 2200 0    60   Input ~ 0
-BDAL7
-Text GLabel 14150 2300 0    60   Input ~ 0
-BDAL8
-Text GLabel 14150 2400 0    60   Input ~ 0
-BDAL9
-Text GLabel 14150 2500 0    60   Input ~ 0
-BDAL10
-Text GLabel 14150 2600 0    60   Input ~ 0
-BDAL11
-Text GLabel 14150 2700 0    60   Input ~ 0
-BDAL12
-Text GLabel 14150 2800 0    60   Input ~ 0
-BDAL13
-Text GLabel 14150 2900 0    60   Input ~ 0
-BDAL14
-Text GLabel 14150 3000 0    60   Input ~ 0
-BDAL15
-Text GLabel 14150 3100 0    60   Input ~ 0
-BDAL16
-Text GLabel 14150 3200 0    60   Input ~ 0
-BDAL17
-Text GLabel 14150 3300 0    60   Input ~ 0
-BDAL18
-Text GLabel 14150 3400 0    60   Input ~ 0
-BDAL19
-Text GLabel 14150 3500 0    60   Input ~ 0
-BDAL20
-Text GLabel 14150 3600 0    60   Input ~ 0
-BDAL21
-Text GLabel 14150 3750 0    60   Input ~ 0
-BBS7
-Text GLabel 14150 3850 0    60   Input ~ 0
-BSYNC
-Text GLabel 14150 3950 0    60   Input ~ 0
-BDIN
-Text GLabel 14150 4150 0    60   Input ~ 0
-BRPLY
-Text GLabel 14150 4250 0    60   Input ~ 0
-BWTBT
-Text GLabel 14150 4350 0    60   Input ~ 0
-BREF
-Text GLabel 14150 4500 0    60   Input ~ 0
-BHALT
-Text GLabel 14150 4600 0    60   Input ~ 0
-BINIT
-Text GLabel 14150 4750 0    60   Input ~ 0
-BDMR
-Text GLabel 14150 5200 0    60   Input ~ 0
-BIRQ4
-Text GLabel 14150 5300 0    60   Input ~ 0
-BIRQ5
-Text GLabel 14150 5400 0    60   Input ~ 0
-BIRQ6
-Text GLabel 14150 5500 0    60   Input ~ 0
-BIRQ7
-Text GLabel 14150 5600 0    60   Input ~ 0
-BIAKI
-Text GLabel 14150 5700 0    60   Input ~ 0
-BIAKO
-Text GLabel 14150 5800 0    60   Input ~ 0
-BEVNT
-Text GLabel 15800 3350 2    60   Input ~ 0
-BPOK
-Text GLabel 15800 3450 2    60   Input ~ 0
-BDCOK
-Wire Notes Line
-	13550 1750 13550 5100
-Wire Notes Line
-	13550 5100 12600 5100
-Wire Wire Line
-	15800 4300 15900 4300
-Wire Wire Line
-	15900 4300 15900 5000
-Wire Wire Line
-	15800 4900 15900 4900
-Connection ~ 15900 4900
-Wire Wire Line
-	15800 4800 15900 4800
-Connection ~ 15900 4800
-Wire Wire Line
-	15800 4700 15900 4700
-Connection ~ 15900 4700
-Wire Wire Line
-	15800 4600 15900 4600
-Connection ~ 15900 4600
-Wire Wire Line
-	15800 4500 15900 4500
-Connection ~ 15900 4500
-Wire Wire Line
-	15800 4400 15900 4400
-Connection ~ 15900 4400
 $Comp
-L GND #PWR01
-U 1 1 56137AAE
-P 15900 5000
-F 0 "#PWR01" H 15900 4750 50  0001 C CNN
-F 1 "GND" H 15900 4850 50  0000 C CNN
-F 2 "" H 15900 5000 60  0000 C CNN
-F 3 "" H 15900 5000 60  0000 C CNN
-	1    15900 5000
-	1    0    0    -1
-$EndComp
-$Comp
-L +5V #PWR02
-U 1 1 56137AC5
-P 15900 4000
-F 0 "#PWR02" H 15900 3850 50  0001 C CNN
-F 1 "+5V" H 15900 4140 50  0000 C CNN
-F 2 "" H 15900 4000 60  0000 C CNN
-F 3 "" H 15900 4000 60  0000 C CNN
-	1    15900 4000
-	0    1    1    0
-$EndComp
-Wire Wire Line
-	15800 4000 15900 4000
-Wire Wire Line
-	15800 4100 15900 4100
-Wire Wire Line
-	15900 4000 15900 4200
-Wire Wire Line
-	15900 4200 15800 4200
-Connection ~ 15900 4100
-$Comp
-L PWR_FLAG #FLG03
+L PWR_FLAG #FLG01
 U 1 1 56137D79
 P 15350 6350
-F 0 "#FLG03" H 15350 6445 50  0001 C CNN
+F 0 "#FLG01" H 15350 6445 50  0001 C CNN
 F 1 "PWR_FLAG" H 15350 6530 50  0000 C CNN
 F 2 "" H 15350 6350 60  0000 C CNN
@@
 $EndComp
 $Comp
-L PWR_FLAG #FLG04
+L PWR_FLAG #FLG02
 U 1 1 56137D87
 P 15800 6350
-F 0 "#FLG04" H 15800 6445 50  0001 C CNN
+F 0 "#FLG02" H 15800 6445 50  0001 C CNN
 F 1 "PWR_FLAG" H 15800 6530 50  0000 C CNN
 F 2 "" H 15800 6350 60  0000 C CNN
@@
 $EndComp
 $Comp
-L +5V #PWR05
+L +5V #PWR03
 U 1 1 56137DA4
 P 15350 6350
-F 0 "#PWR05" H 15350 6200 50  0001 C CNN
+F 0 "#PWR03" H 15350 6200 50  0001 C CNN
 F 1 "+5V" H 15350 6490 50  0000 C CNN
 F 2 "" H 15350 6350 60  0000 C CNN
@@
 $EndComp
 $Comp
-L GND #PWR06
+L GND #PWR04
 U 1 1 56137DB2
 P 15800 6350
-F 0 "#PWR06" H 15800 6100 50  0001 C CNN
+F 0 "#PWR04" H 15800 6100 50  0001 C CNN
 F 1 "GND" H 15800 6200 50  0000 C CNN
 F 2 "" H 15800 6350 60  0000 C CNN
@@
 	1    0    0    -1
 $EndComp
-Text GLabel 14150 4050 0    60   Input ~ 0
-BDOUT
-NoConn ~ 15800 3600
-NoConn ~ 15800 3700
-NoConn ~ 15800 3800
-NoConn ~ 15800 3900
-NoConn ~ 15800 3250
-NoConn ~ 15800 3150
-NoConn ~ 15800 3050
-NoConn ~ 15800 2950
-NoConn ~ 15800 2850
-NoConn ~ 15800 2300
-NoConn ~ 15800 2200
-NoConn ~ 15800 2100
-NoConn ~ 15800 2000
-NoConn ~ 15800 1900
-NoConn ~ 15800 1800
 $EndSCHEMATC

Commit message: Changed to comparator for bus receivers and rearranged schematic to multiple pages
Parts:
- added B101: QBUS, myMods.pretty:Qbus-double, symbol QBUS
Connections:
- net labels added: +12V, BBS7, BDAL0, BDAL1, BDAL10, BDAL11, BDAL12, BDAL13, BDAL14, BDAL15, BDAL16, BDAL17, BDAL18, BDAL19, BDAL2, BDAL20, BDAL21, BDAL3, BDAL4, BDAL5, BDAL6, BDAL7, BDAL8, BDAL9, BDCOK, BDIN, BDMGI, BDMGO, BDMR, BDOUT, BEVNT, BHALT, BIAKI, BIAKO, BINIT, BIRQ4, BIRQ5, BIRQ6, BIRQ7, BPOK, BREF, BRPLY, BSACK, BSYNC, BWTBT
- wire segments 0 -> 15
- no-connect marks 0 -> 13

Commit message: Added the FPGA and rearranged the sheets.
Parts:
- added U401: XC7A75T-CSG324, myMods.pretty:CSG324, symbol XC7A75T-CSG324
Connections:
- net labels added: BDAL[0..21], RBS7, RDAL[0..21], RDCOK, RDIN, RDMGI, RDMR, RDOUT, REVNT, RHALT, RIAKI, RINIT, RIRQ4, RIRQ5, RIRQ6, RIRQ7, RPOK, RREF, RRPLY, RSACK, RSYNC, RWTBT, TBS7, TDAL[0..21], TDIN, TDMGO, TDMR, TDOUT, TIAKO, TINIT, TIRQ4, TIRQ5, TIRQ6, TIRQ7, TREF, TRPLY, TSACK, TSYNC, TWTBT
- net labels removed: BBS7, BDCOK, BDIN, BDMGI, BDMGO, BDMR, BDOUT, BEVNT, BHALT, BIAKI, BIAKO, BINIT, BIRQ4, BIRQ5, BIRQ6, BIRQ7, BPOK, BREF, BRPLY, BSACK, BSYNC, BWTBT
- wire segments 15 -> 71

Commit message: Updated to KiCad v5
Parts:
- B101: symbol QBUS -> myLib:QBUS
- U401: symbol XC7A75T-CSG324 -> myLib:XC7A75T-CSG324
Connections:
- wire segments 71 -> 80
Changed lines of the file:
@@
-EESchema Schematic File Version 2
-LIBS:qsic-rescue
-LIBS:power
-LIBS:device
-LIBS:transistors
-LIBS:conn
-LIBS:linear
-LIBS:regul
-LIBS:74xx
-LIBS:cmos4000
-LIBS:adc-dac
-LIBS:memory
-LIBS:xilinx
-LIBS:microcontrollers
-LIBS:dsp
-LIBS:microchip
-LIBS:analog_switches
-LIBS:motorola
-LIBS:texas
-LIBS:intel
-LIBS:audio
-LIBS:interface
-LIBS:digital-audio
-LIBS:philips
-LIBS:display
-LIBS:cypress
-LIBS:siliconi
-LIBS:opto
-LIBS:atmel
-LIBS:contrib
-LIBS:valves
-LIBS:myLib
+EESchema Schematic File Version 4
 LIBS:qsic-cache
-EELAYER 25 0
+EELAYER 26 0
 EELAYER END
 $Descr A 11000 8500
@@
 $EndDescr
 $Comp
-L PWR_FLAG #FLG01
+L power:PWR_FLAG #FLG01
 U 1 1 56137D79
 P 5000 7500
@@
 $EndComp
 $Comp
-L PWR_FLAG #FLG02
+L power:PWR_FLAG #FLG02
 U 1 1 56137D87
 P 5400 7500
@@
 $EndComp
 $Comp
-L +5V #PWR03
+L power:+5V #PWR03
 U 1 1 56137DA4
 P 5000 7500
@@
 $EndComp
 $Comp
-L GND #PWR04
+L power:GND #PWR04
 U 1 1 56137DB2
 P 5400 7500
@@
 $EndComp
 $Comp
-L GND #PWR05
+L power:GND #PWR05
 U 1 1 58814E97
 P 900 5000
@@
 $EndComp
 $Comp
-L +5V #PWR06
+L power:+5V #PWR06
 U 1 1 58814E9D
 P 850 4000
@@
 NoConn ~ 1000 1800
 $Comp
-L QBUS B101
+L myLib:QBUS B101
 U 1 1 58814EB8
 P 1200 3600
@@
 $EndComp
 $Comp
-L +12V #PWR07
+L power:+12V #PWR07
 U 1 1 58814ECD
 P 850 3600
@@
 $EndComp
 $Comp
-L PWR_FLAG #FLG08
+L power:PWR_FLAG #FLG08
 U 1 1 58814F6A
 P 5800 7500
@@
 $EndComp
 $Comp
-L +12V #PWR09
+L power:+12V #PWR09
 U 1 1 58814F79
 P 5800 7500
@@
 $EndSheet
 $Comp
-L XC7A75T-CSG324 U401
+L myLib:XC7A75T-CSG324 U401
 U 4 1 58C75923
 P 7900 5800
@@
 $EndComp
 $Comp
-L XC7A75T-CSG324 U401
+L myLib:XC7A75T-CSG324 U401
 U 5 1 58C75986
 P 10300 5800
@@
 	1000 4300 900  4300
 Wire Wire Line
-	900  4300 900  5000
+	900  4300 900  4400
 Wire Wire Line
 	1000 4900 900  4900
@@
 Connection ~ 900  4400
 Wire Wire Line
-	850  4000 1000 4000
+	850  4000 900  4000
 Wire Wire Line
 	1000 4100 900  4100
 Wire Wire Line
-	900  4000 900  4200
+	900  4000 900  4100
 Wire Wire Line
 	900  4200 1000 4200
 Connection ~ 900  4100
 Wire Wire Line
-	850  3600 1000 3600
+	850  3600 900  3600
 Wire Wire Line
 	1000 3700 900  3700
@@
 Wire Wire Line
 	2650 3600 3000 3600
-Wire Bus Line
-	3100 1350 3100 3700
 Wire Bus Line
 	3650 1350 3100 1350
@@
 F1 "io.sch" 60
 $EndSheet
+Wire Wire Line
+	900  4900 900  5000
+Wire Wire Line
+	900  4800 900  4900
+Wire Wire Line
+	900  4700 900  4800
+Wire Wire Line
+	900  4600 900  4700
+Wire Wire Line
+	900  4500 900  4600
+Wire Wire Line
+	900  4400 900  4500
+Wire Wire Line
+	900  4100 900  4200
+Wire Wire Line
+	900  3600 1000 3600
+Wire Wire Line
+	900  4000 1000 4000
+Wire Bus Line
+	3100 1350 3100 3700
 $EndSCHEMATC

Commit message: Updated to KiCad v5
Parts:
- U401: symbol myLib:XC7A75T-CSG324 -> qsic-rescue:XC7A75T-CSG324-myLib
Changed lines of the file:
@@
 EESchema Schematic File Version 4
 LIBS:qsic-cache
-EELAYER 26 0
+EELAYER 30 0
 EELAYER END
 $Descr A 11000 8500
 encoding utf-8
-Sheet 1 6
+Sheet 1 7
 Title "QBUS Interface"
 Date "2017-10-31"
@@
 $EndSheet
 $Comp
-L myLib:XC7A75T-CSG324 U401
+L qsic-rescue:XC7A75T-CSG324-myLib U401
 U 4 1 58C75923
 P 7900 5800
@@
 $EndComp
 $Comp
-L myLib:XC7A75T-CSG324 U401
+L qsic-rescue:XC7A75T-CSG324-myLib U401
 U 5 1 58C75986
 P 10300 5800
