File: board-smt/xcvr.sch (KiCad schematic (older format))
At the start: 5 parts

Commit message: These are all old changes in directories that are now historical.
Parts:
- R360, R372, R373: renamed from R?; footprint Resistors_SMD:R_0603 -> Resistor_SMD:R_0603_1608Metric; symbol qsic-rescue:R-device -> Device:R_US
- gave numbers to parts that had none: 2
Connections:
- net Bus: now also Q307.3 (D); no longer Q307.6 (D)
- net GND: now also Q307.4 (S); no longer Q307.1 (S)
- net at R360.1: now also Q307.5 (G); no longer Q307.2 (G)
Changed lines of the file:
@@
 EESchema Schematic File Version 4
-LIBS:qsic-cache
 EELAYER 30 0
 EELAYER END
 $Descr A 11000 8500
 encoding utf-8
-Sheet 3 7
+Sheet 3 8
 Title "Bus Transceiver"
 Date ""
@@
 $EndDescr
 $Comp
-L myLib:Dual_NMOS Q?
-U 1 1 5CBC3826
+L myLib:Dual_NMOS Q307
+U 2 1 5CBC3826
 P 5025 3700
-F 0 "Q?" H 4975 3600 50  0000 R CNN
+F 0 "Q307" H 4975 3600 50  0000 R CNN
 F 1 "Dual_NMOS" H 5025 3500 50  0000 R CNN
 F 2 "TO_SOT_Packages_SMD:SOT-23-6" H 5225 3800 29  0001 C CNN
 F 3 "" H 5025 3700 60  0000 C CNN
-	1    5025 3700
+	2    5025 3700
 	1    0    0    -1
 $EndComp
 $Comp
-L qsic-rescue:R-device R?
+L Device:R_US R360
 U 1 1 5CBC382D
 P 4625 3700
-F 0 "R?" V 4705 3700 50  0000 C CNN
-F 1 "R" V 4625 3700 50  0000 C CNN
-F 2 "Resistors_SMD:R_0603" V 4555 3700 30  0001 C CNN
+F 0 "R360" V 4705 3700 50  0000 C CNN
+F 1 "R" V 4525 3700 50  0000 C CNN
+F 2 "Resistor_SMD:R_0603_1608Metric" V 4555 3700 30  0001 C CNN
 F 3 "" H 4625 3700 30  0000 C CNN
 	1    4625 3700
@@
 $EndComp
 $Comp
-L power:GND #PWR?
+L power:GND #PWR0163
 U 1 1 5CBC3834
 P 5125 3900
-F 0 "#PWR?" H 5125 3650 50  0001 C CNN
+F 0 "#PWR0163" H 5125 3650 50  0001 C CNN
 F 1 "GND" H 5125 3750 50  0001 C CNN
 F 2 "" H 5125 3900 60  0000 C CNN
@@
 $EndComp
 $Comp
-L qsic-rescue:R-device R?
+L Device:R_US R?
 U 1 1 5CBC383A
 P 5050 3200
 AR Path="/58857B5F/5CBC383A" Ref="R?"  Part="1"
-AR Path="/58857B5F/5CBC325F/5CBC383A" Ref="R?"  Part="1"
-F 0 "R?" V 5130 3200 50  0000 C CNN
-F 1 "20kΩ" V 5050 3200 50  0000 C CNN
-F 2 "Resistors_SMD:R_0603" V 4980 3200 50  0001 C CNN
+AR Path="/58857B5F/5CBC325F/5CBC383A" Ref="R372"  Part="1"
+F 0 "R372" V 5130 3200 50  0000 C CNN
+F 1 "20kΩ" V 4950 3200 50  0000 C CNN
+F 2 "Resistor_SMD:R_0603_1608Metric" V 4980 3200 50  0001 C CNN
 F 3 "" H 5050 3200 50  0000 C CNN
 	1    5050 3200
@@
 $EndComp
 $Comp
-L qsic-rescue:R-device R?
+L Device:R_US R373
 U 1 1 5CBC3841
 P 5675 3200
-F 0 "R?" V 5755 3200 50  0000 C CNN
-F 1 "340kΩ" V 5675 3200 50  0000 C CNN
-F 2 "Resistors_SMD:R_0603" V 5605 3200 50  0001 C CNN
+F 0 "R373" V 5755 3200 50  0000 C CNN
+F 1 "340kΩ" V 5575 3200 50  0000 C CNN
+F 2 "Resistor_SMD:R_0603_1608Metric" V 5605 3200 50  0001 C CNN
 F 3 "" H 5675 3200 50  0000 C CNN
 	1    5675 3200
@@
 $EndComp
 $Comp
-L myLib:CMP401 U?
+L myLib:CMP401 U310
 U 3 1 5CBC3848
 P 5525 3400
-F 0 "U?" H 6025 3500 60  0000 C CNN
+F 0 "U310" H 6025 3500 60  0000 C CNN
 F 1 "CMP401" H 6125 3200 60  0000 C CNN
 F 2 "Housings_SOIC:SOIC-16_3.9x9.9mm_Pitch1.27mm" H 5525 3400 60  0001 C CNN
